File: expansion.kicad_sch (KiCad schematic)
At the start: 4 parts, among them P1 EXPANSION BUS

Commit message: cleaned up side connector footprint to get rid of DRC errors
Parts:
- P1: footprint Raemixx500:A2000_COPRO_SLOT -> Raemixx500:A500_SIDE_SLOT
Changed lines of the file:
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@@
 			)
 		)
-		(property "Footprint" "Raemixx500:A2000_COPRO_SLOT"
+		(property "Footprint" "Raemixx500:A500_SIDE_SLOT"
 			(at 145.161 91.44 0)
 			(effects

Commit message: DRAM chips replaced with SIMM module
Added logic to decode 2MB chip + 1.5MB slow
Rewired trapdoor slot
Other:
- title: Rämixx500 -> Rämixx500_max
Changed lines of the file:
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@@
 	(paper "A4")
 	(title_block
-		(title "Rämixx500")
-		(date "2019-06-23")
-		(rev "1")
+		(title "Rämixx500_max")
+		(date "2026-03-13")
+		(rev "2")
 		(company "SukkoPera")
 		(comment 4 "Licensed under CC BY-NC-SA 4.0")

Commit message: Started cleaning up BOM
Parts:
- P1: now left out of the parts list
Changed lines of the file:
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@@
 		(unit 1)
 		(exclude_from_sim no)
-		(in_bom yes)
+		(in_bom no)
 		(on_board yes)
 		(dnp no)

Commit message: more work on BOM done
Parts:
- E702, E703, E704: Mouser (none) -> 81-DSS1NB32A103Q91A
Changed lines of the file:
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@@
 			)
 		)
-		(property "Mouser" ""
+		(property "Mouser" " 81-DSS1NB32A103Q91A "
 			(at 197.231 25.908 0)
 			(effects
@@
 			)
 		)
-		(property "Mouser" ""
+		(property "Mouser" " 81-DSS1NB32A103Q91A "
 			(at 197.231 41.91 0)
 			(effects
@@
 			)
 		)
-		(property "Mouser" ""
-			(at 197.231 50.8 0)
-			(effects
+		(property "Mouser" " 81-DSS1NB32A103Q91A "
+			(at 197.231 50.8 0)
+			(effects
