File: expansion.kicad_sch (KiCad schematic)
At the start: 4 parts, among them P1 EXPANSION BUS

Commit message: More BOM work
I am marking optional components as DNP to get some overview
Parts:
- E702, E703, E704: Mouser 81-DSS1NB32A103Q91A -> 81-DSS1NB32A103Q91A
Changed lines of the file:
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@@
 			)
 		)
-		(property "Mouser" " 81-DSS1NB32A103Q91A "
+		(property "Mouser" "81-DSS1NB32A103Q91A "
 			(at 197.231 25.908 0)
 			(effects
@@
 			)
 		)
-		(property "Mouser" " 81-DSS1NB32A103Q91A "
+		(property "Mouser" "81-DSS1NB32A103Q91A "
 			(at 197.231 41.91 0)
 			(effects
@@
 			)
 		)
-		(property "Mouser" " 81-DSS1NB32A103Q91A "
-			(at 197.231 50.8 0)
-			(effects
+		(property "Mouser" "81-DSS1NB32A103Q91A "
+			(at 197.231 50.8 0)
+			(effects
