File: clockdist.kicad_sch (KiCad schematic)
At the start: 16 parts, among them U33 74LS258

Commit message: DRAM chips replaced with SIMM module
Added logic to decode 2MB chip + 1.5MB slow
Rewired trapdoor slot
Other:
- title: Rämixx500 -> Rämixx500_max
Changed lines of the file:
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@@
 	(paper "A4")
 	(title_block
-		(title "Rämixx500")
-		(date "2019-04-20")
-		(rev "1")
+		(title "Rämixx500_max")
+		(date "2026-03-13")
+		(rev "2")
 		(company "SukkoPera")
 		(comment 4 "Licensed under CC BY-NC-SA 4.0")

Commit message: Working on BOM
Parts:
- C33: MFG Part Num C410C103K1H5TAAUTO -> C410C103K1R5TA; Mouser (none) -> 80-C410C103K1R
Changed lines of the file:
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@@
+			)
+		)
+		(property "Mouser" ""
+			(at 155.194 121.158 0)
+			(effects
+				(font
+					(size 1.27 1.27)
+				)
+				(hide yes)
 			)
 		)
@@
 			)
 		)
+		(property "Mouser" ""
+			(at 166.37 121.412 0)
+			(effects
+				(font
+					(size 1.27 1.27)
+				)
+				(hide yes)
+			)
+		)
 		(pin "2"
 		)
@@
 			)
 		)
+		(property "Mouser" ""
+			(at 177.546 121.412 0)
+			(effects
+				(font
+					(size 1.27 1.27)
+				)
+				(hide yes)
+			)
+		)
 		(pin "1"
 		)
@@
 			)
 		)
+		(property "Mouser" ""
+			(at 188.722 121.666 0)
+			(effects
+				(font
+					(size 1.27 1.27)
+				)
+				(hide yes)
+			)
+		)
 		(pin "1"
 		)
@@
 			)
 		)
+		(property "Mouser" ""
+			(at 199.898 121.666 0)
+			(effects
+				(font
+					(size 1.27 1.27)
+				)
+				(hide yes)
+			)
+		)
 		(pin "1"
 		)
@@
 			)
 		)
+		(property "Mouser" ""
+			(at 50.8 120.904 0)
+			(effects
+				(font
+					(size 1.27 1.27)
+				)
+				(hide yes)
+			)
+		)
 		(pin "2"
 		)
@@
 			)
 		)
+		(property "Mouser" ""
+			(at 61.976 121.158 0)
+			(effects
+				(font
+					(size 1.27 1.27)
+				)
+				(hide yes)
+			)
+		)
 		(pin "1"
 		)
@@
 			)
 		)
+		(property "Mouser" ""
+			(at 73.152 121.158 0)
+			(effects
+				(font
+					(size 1.27 1.27)
+				)
+				(hide yes)
+			)
+		)
 		(pin "1"
 		)
@@
 			)
 		)
+		(property "Mouser" ""
+			(at 61.976 172.466 0)
+			(effects
+				(font
+					(size 1.27 1.27)
+				)
+				(hide yes)
+			)
+		)
 		(pin "1"
 		)
@@
 			)
 		)
+		(property "Mouser" ""
+			(at 73.152 172.72 0)
+			(effects
+				(font
+					(size 1.27 1.27)
+				)
+				(hide yes)
+			)
+		)
 		(pin "1"
 		)
@@
 			)
 		)
+		(property "Mouser" ""
+			(at 136.906 102.87 0)
+			(effects
+				(font
+					(size 1.27 1.27)
+				)
+				(hide yes)
+			)
+		)
 		(pin "1"
 		)
@@
 			)
 		)
+		(property "Mouser" ""
+			(at 136.906 113.03 0)
+			(effects
+				(font
+					(size 1.27 1.27)
+				)
+				(hide yes)
+			)
+		)
 		(pin "3"
 		)
@@
 			)
 		)
+		(property "Mouser" ""
+			(at 92.456 64.77 0)
+			(effects
+				(font
+					(size 1.27 1.27)
+				)
+				(hide yes)
+			)
+		)
 		(pin "15"
 		)
@@
 			)
 		)
+		(property "Mouser" ""
+			(at 92.456 100.33 0)
+			(effects
+				(font
+					(size 1.27 1.27)
+				)
+				(hide yes)
+			)
+		)
 		(pin "1"
 		)
@@
 			)
 		)
+		(property "Mouser" ""
+			(at 92.456 82.55 0)
+			(effects
+				(font
+					(size 1.27 1.27)
+				)
+				(hide yes)
+			)
+		)
 		(pin "5"
 		)
@@
 			)
 		)
+		(property "Mouser" ""
+			(at 133.096 82.55 90)
+			(effects
+				(font
+					(size 1.27 1.27)
+				)
+				(hide yes)
+			)
+		)
 		(pin "3"
 		)
@@
 			)
 		)
+		(property "Mouser" ""
+			(at 248.666 95.758 0)
+			(effects
+				(font
+					(size 1.27 1.27)
+				)
+				(hide yes)
+			)
+		)
 		(pin "2"
 		)
@@
 			)
 		)
+		(property "Mouser" ""
+			(at 246.126 72.898 90)
+			(effects
+				(font
+					(size 1.27 1.27)
+				)
+				(hide yes)
+			)
+		)
 		(pin "2"
 		)
@@
 			)
 		)
-		(property "MFG Part Num" "C410C103K1H5TAAUTO"
+		(property "MFG Part Num" "C410C103K1R5TA "
 			(at 258.826 98.298 0)
 			(effects
@@
 			(at 258.826 98.298 0)
 			(effects
+				(font
+					(size 1.27 1.27)
+				)
+				(hide yes)
+			)
+		)
+		(property "Mouser" "80-C410C103K1R"
+			(at 258.826 98.298 0)
+			(effects

Commit message: more work on BOM done
Parts:
- E102, E103, E106, E107, E108: MFG Name (none) -> VISHAY; MFG Part Num (none) -> A470J15C0GF5TAA; Mouser (none) -> 594-A470J15C0GF5TAA
- E104, E105: MFG Name (none) -> YAGEO; MFG Part Num (none) -> MFR-25FBF52-68R; Mouser (none) -> 603-MFR-25FBF52-68R
- E407: Mouser (none) -> 81-DSS1NB32A103Q91A
Changed lines of the file:
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@@
 			)
 		)
-		(property "Mouser" ""
+		(property "Mouser" "594-A470J15C0GF5TAA"
+			(at 199.898 121.666 0)
+			(effects
+				(font
+					(size 1.27 1.27)
+				)
+				(hide yes)
+			)
+		)
+		(property "MFG Name" "VISHAY"
+			(at 199.898 121.666 0)
+			(effects
+				(font
+					(size 1.27 1.27)
+				)
+				(hide yes)
+			)
+		)
+		(property "MFG Part Num" "A470J15C0GF5TAA "
 			(at 199.898 121.666 0)
 			(effects
@@
 			)
 		)
-		(property "Mouser" ""
+		(property "Mouser" "594-A470J15C0GF5TAA"
+			(at 50.8 120.904 0)
+			(effects
+				(font
+					(size 1.27 1.27)
+				)
+				(hide yes)
+			)
+		)
+		(property "MFG Name" "VISHAY"
+			(at 50.8 120.904 0)
+			(effects
+				(font
+					(size 1.27 1.27)
+				)
+				(hide yes)
+			)
+		)
+		(property "MFG Part Num" "A470J15C0GF5TAA "
 			(at 50.8 120.904 0)
 			(effects
@@
 			)
 		)
-		(property "Mouser" ""
+		(property "Mouser" "594-A470J15C0GF5TAA"
+			(at 61.976 121.158 0)
+			(effects
+				(font
+					(size 1.27 1.27)
+				)
+				(hide yes)
+			)
+		)
+		(property "MFG Name" "VISHAY"
+			(at 61.976 121.158 0)
+			(effects
+				(font
+					(size 1.27 1.27)
+				)
+				(hide yes)
+			)
+		)
+		(property "MFG Part Num" "A470J15C0GF5TAA "
 			(at 61.976 121.158 0)
 			(effects
@@
 			)
 		)
-		(property "Mouser" ""
+		(property "Mouser" "594-A470J15C0GF5TAA"
+			(at 73.152 121.158 0)
+			(effects
+				(font
+					(size 1.27 1.27)
+				)
+				(hide yes)
+			)
+		)
+		(property "MFG Name" "VISHAY"
+			(at 73.152 121.158 0)
+			(effects
+				(font
+					(size 1.27 1.27)
+				)
+				(hide yes)
+			)
+		)
+		(property "MFG Part Num" "A470J15C0GF5TAA "
 			(at 73.152 121.158 0)
 			(effects
@@
 			)
 		)
-		(property "Mouser" ""
+		(property "Mouser" "594-A470J15C0GF5TAA"
+			(at 73.152 172.72 0)
+			(effects
+				(font
+					(size 1.27 1.27)
+				)
+				(hide yes)
+			)
+		)
+		(property "MFG Name" "VISHAY"
+			(at 73.152 172.72 0)
+			(effects
+				(font
+					(size 1.27 1.27)
+				)
+				(hide yes)
+			)
+		)
+		(property "MFG Part Num" "A470J15C0GF5TAA "
 			(at 73.152 172.72 0)
 			(effects
@@
 			)
 		)
-		(property "Mouser" ""
+		(property "Mouser" "603-MFR-25FBF52-68R "
+			(at 136.906 102.87 0)
+			(effects
+				(font
+					(size 1.27 1.27)
+				)
+				(hide yes)
+			)
+		)
+		(property "MFG Name" "YAGEO"
+			(at 136.906 102.87 0)
+			(effects
+				(font
+					(size 1.27 1.27)
+				)
+				(hide yes)
+			)
+		)
+		(property "MFG Part Num" "MFR-25FBF52-68R "
 			(at 136.906 102.87 0)
 			(effects
@@
 			)
 		)
-		(property "Mouser" ""
+		(property "Mouser" "603-MFR-25FBF52-68R "
+			(at 136.906 113.03 0)
+			(effects
+				(font
+					(size 1.27 1.27)
+				)
+				(hide yes)
+			)
+		)
+		(property "MFG Name" "YAGEO"
+			(at 136.906 113.03 0)
+			(effects
+				(font
+					(size 1.27 1.27)
+				)
+				(hide yes)
+			)
+		)
+		(property "MFG Part Num" "MFR-25FBF52-68R "
 			(at 136.906 113.03 0)
 			(effects
@@
 			)
 		)
-		(property "Mouser" ""
+		(property "Mouser" " 81-DSS1NB32A103Q91A "
 			(at 246.126 72.898 90)
 			(effects

Commit message: More BOM work
I am marking optional components as DNP to get some overview
Parts:
- E109, E791, E792, E793, E794: MFG Name (none) -> VISHAY; MFG Part Num (none) -> A470J15C0GF5TAA; Mouser (none) -> 594-A470J15C0GF5TAA
- E407: Mouser 81-DSS1NB32A103Q91A -> 81-DSS1NB32A103Q91A
Changed lines of the file:
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@@
 			)
 		)
-		(property "Mouser" ""
+		(property "Mouser" "594-A470J15C0GF5TAA"
+			(at 155.194 121.158 0)
+			(effects
+				(font
+					(size 1.27 1.27)
+				)
+				(hide yes)
+			)
+		)
+		(property "MFG Name" "VISHAY"
+			(at 155.194 121.158 0)
+			(effects
+				(font
+					(size 1.27 1.27)
+				)
+				(hide yes)
+			)
+		)
+		(property "MFG Part Num" "A470J15C0GF5TAA "
 			(at 155.194 121.158 0)
 			(effects
@@
 			)
 		)
-		(property "Mouser" ""
+		(property "Mouser" "594-A470J15C0GF5TAA"
+			(at 166.37 121.412 0)
+			(effects
+				(font
+					(size 1.27 1.27)
+				)
+				(hide yes)
+			)
+		)
+		(property "MFG Name" "VISHAY"
+			(at 166.37 121.412 0)
+			(effects
+				(font
+					(size 1.27 1.27)
+				)
+				(hide yes)
+			)
+		)
+		(property "MFG Part Num" "A470J15C0GF5TAA "
 			(at 166.37 121.412 0)
 			(effects
@@
 			)
 		)
-		(property "Mouser" ""
+		(property "Mouser" "594-A470J15C0GF5TAA"
+			(at 177.546 121.412 0)
+			(effects
+				(font
+					(size 1.27 1.27)
+				)
+				(hide yes)
+			)
+		)
+		(property "MFG Name" "VISHAY"
+			(at 177.546 121.412 0)
+			(effects
+				(font
+					(size 1.27 1.27)
+				)
+				(hide yes)
+			)
+		)
+		(property "MFG Part Num" "A470J15C0GF5TAA "
 			(at 177.546 121.412 0)
 			(effects
@@
 			)
 		)
-		(property "Mouser" ""
+		(property "Mouser" "594-A470J15C0GF5TAA"
+			(at 188.722 121.666 0)
+			(effects
+				(font
+					(size 1.27 1.27)
+				)
+				(hide yes)
+			)
+		)
+		(property "MFG Name" "VISHAY"
+			(at 188.722 121.666 0)
+			(effects
+				(font
+					(size 1.27 1.27)
+				)
+				(hide yes)
+			)
+		)
+		(property "MFG Part Num" "A470J15C0GF5TAA "
 			(at 188.722 121.666 0)
 			(effects
@@
 			)
 		)
-		(property "Mouser" ""
+		(property "Mouser" "594-A470J15C0GF5TAA"
+			(at 61.976 172.466 0)
+			(effects
+				(font
+					(size 1.27 1.27)
+				)
+				(hide yes)
+			)
+		)
+		(property "MFG Name" "VISHAY"
+			(at 61.976 172.466 0)
+			(effects
+				(font
+					(size 1.27 1.27)
+				)
+				(hide yes)
+			)
+		)
+		(property "MFG Part Num" "A470J15C0GF5TAA "
 			(at 61.976 172.466 0)
 			(effects
@@
 			)
 		)
-		(property "Mouser" " 81-DSS1NB32A103Q91A "
+		(property "Mouser" "81-DSS1NB32A103Q91A "
 			(at 246.126 72.898 90)
 			(effects

Commit message: BOM updates
Parts:
- RP103: MFG Name (none) -> BOURNS; MFG Part Num (none) -> 4610X-102-390LF; Mouser (none) -> 652-4610X-2LF-39
- U33: MFG Name N/A -> TI; MFG Part Num (none) -> SN74LS258BN; Mouser (none) -> 595-SN74LS258BN
Changed lines of the file:
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@@
 			)
 		)
-		(property "MFG Name" "N/A"
+		(property "MFG Name" "TI"
 			(at 92.456 64.77 0)
 			(effects
@@
 			)
 		)
-		(property "Mouser" ""
+		(property "Mouser" "595-SN74LS258BN "
+			(at 92.456 64.77 0)
+			(effects
+				(font
+					(size 1.27 1.27)
+				)
+				(hide yes)
+			)
+		)
+		(property "MFG Part Num" "SN74LS258BN"
 			(at 92.456 64.77 0)
 			(effects
@@
 			)
 		)
-		(property "MFG Name" "N/A"
+		(property "MFG Name" "TI"
 			(at 92.456 100.33 0)
 			(effects
@@
 			)
 		)
-		(property "Mouser" ""
+		(property "Mouser" "595-SN74LS258BN "
+			(at 92.456 100.33 0)
+			(effects
+				(font
+					(size 1.27 1.27)
+				)
+				(hide yes)
+			)
+		)
+		(property "MFG Part Num" "SN74LS258BN"
 			(at 92.456 100.33 0)
 			(effects
@@
 			)
 		)
-		(property "MFG Name" "N/A"
+		(property "MFG Name" "TI"
 			(at 92.456 82.55 0)
 			(effects
@@
 			)
 		)
-		(property "Mouser" ""
+		(property "Mouser" "595-SN74LS258BN "
+			(at 92.456 82.55 0)
+			(effects
+				(font
+					(size 1.27 1.27)
+				)
+				(hide yes)
+			)
+		)
+		(property "MFG Part Num" "SN74LS258BN"
 			(at 92.456 82.55 0)
 			(effects
@@
 			)
 		)
-		(property "Mouser" ""
+		(property "Mouser" "652-4610X-2LF-39"
+			(at 133.096 82.55 90)
+			(effects
+				(font
+					(size 1.27 1.27)
+				)
+				(hide yes)
+			)
+		)
+		(property "MFG Name" "BOURNS"
+			(at 133.096 82.55 90)
+			(effects
+				(font
+					(size 1.27 1.27)
+				)
+				(hide yes)
+			)
+		)
+		(property "MFG Part Num" "4610X-102-390LF"
 			(at 133.096 82.55 90)
 			(effects
@@
 			)
 		)
-		(property "MFG Name" "N/A"
+		(property "MFG Name" "TI"
 			(at 248.666 95.758 0)
 			(effects
@@
 			)
 		)
-		(property "Mouser" ""
+		(property "Mouser" "595-SN74LS258BN "
 			(at 248.666 95.758 0)
 			(effects
+				(font
+					(size 1.27 1.27)
+				)
+				(hide yes)
+			)
+		)
+		(property "MFG Part Num" "SN74LS258BN"
+			(at 248.666 95.758 0)
+			(effects
