File: clockdist.kicad_sch (KiCad schematic)
At the start: 16 parts, among them U33 74LS258

Commit message: even  more BOM work
Parts:
- U33: value 74LS258 -> 74F258; MFG Part Num SN74LS258BN -> (none); Mouser 595-SN74LS258BN -> (none)
Changed lines of the file:
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@@
 			)
 		)
-		(property "Value" "74LS258"
+		(property "Value" "74F258"
 			(at 84.836 69.85 0)
 			(effects
@@
 			)
 		)
-		(property "Mouser" "595-SN74LS258BN "
-			(at 92.456 64.77 0)
-			(effects
-				(font
-					(size 1.27 1.27)
-				)
-				(hide yes)
-			)
-		)
-		(property "MFG Part Num" "SN74LS258BN"
+		(property "Mouser" ""
+			(at 92.456 64.77 0)
+			(effects
+				(font
+					(size 1.27 1.27)
+				)
+				(hide yes)
+			)
+		)
+		(property "MFG Part Num" ""
 			(at 92.456 64.77 0)
 			(effects
@@
 			)
 		)
-		(property "Value" "74LS258"
+		(property "Value" "74F258"
 			(at 84.836 105.41 0)
 			(effects
@@
 			)
 		)
-		(property "Mouser" "595-SN74LS258BN "
+		(property "Mouser" ""
 			(at 92.456 100.33 0)
 			(effects
@@
 			)
 		)
-		(property "MFG Part Num" "SN74LS258BN"
+		(property "MFG Part Num" ""
 			(at 92.456 100.33 0)
 			(effects
@@
 			)
 		)
-		(property "Value" "74LS258"
+		(property "Value" "74F258"
 			(at 84.836 87.63 0)
 			(effects
@@
 			)
 		)
-		(property "Mouser" "595-SN74LS258BN "
+		(property "Mouser" ""
 			(at 92.456 82.55 0)
 			(effects
@@
 			)
 		)
-		(property "MFG Part Num" "SN74LS258BN"
+		(property "MFG Part Num" ""
 			(at 92.456 82.55 0)
 			(effects
@@
 			)
 		)
-		(property "Value" "74LS258"
+		(property "Value" "74F258"
 			(at 249.682 103.886 0)
 			(effects
@@
 			)
 		)
-		(property "Mouser" "595-SN74LS258BN "
+		(property "Mouser" ""
 			(at 248.666 95.758 0)
 			(effects
@@
 			)
 		)
-		(property "MFG Part Num" "SN74LS258BN"
+		(property "MFG Part Num" ""
 			(at 248.666 95.758 0)
 			(effects

Commit message: added mouser part numbers
Parts:
- U33: MFG Part Num (none) -> SN74F258N; Mouser (none) -> 595-SN74F258N
Changed lines of the file:
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@@
 			)
 		)
-		(property "Mouser" ""
+		(property "Mouser" "595-SN74F258N "
 			(at 92.456 64.77 0)
 			(effects
@@
 			)
 		)
-		(property "MFG Part Num" ""
+		(property "MFG Part Num" "SN74F258N "
 			(at 92.456 64.77 0)
 			(effects
@@
 			)
 		)
-		(property "Mouser" ""
+		(property "Mouser" "595-SN74F258N "
 			(at 92.456 100.33 0)
 			(effects
@@
 			)
 		)
-		(property "MFG Part Num" ""
+		(property "MFG Part Num" "SN74F258N "
 			(at 92.456 100.33 0)
 			(effects
@@
 			)
 		)
-		(property "Mouser" ""
+		(property "Mouser" "595-SN74F258N "
 			(at 92.456 82.55 0)
 			(effects
@@
 			)
 		)
-		(property "MFG Part Num" ""
+		(property "MFG Part Num" "SN74F258N "
 			(at 92.456 82.55 0)
 			(effects
@@
 			)
 		)
-		(property "Mouser" ""
+		(property "Mouser" "595-SN74F258N "
 			(at 248.666 95.758 0)
 			(effects
@@
 			)
 		)
-		(property "MFG Part Num" ""
+		(property "MFG Part Num" "SN74F258N "
 			(at 248.666 95.758 0)
 			(effects

Commit message: more silkscreen work
removed sockets for standard IC's
Parts:
- U33: footprint Package_DIP:DIP-16_W7.62mm_Socket_LongPads -> Package_DIP:DIP-16_W7.62mm_LongPads
Changed lines of the file:
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@@
 	(title_block
 		(title "Rämixx500_max")
-		(date "2026-04-09")
+		(date "2026-04-26")
 		(rev "3")
 		(company "SukkoPera")
@@
 			)
 		)
-		(property "Footprint" "Package_DIP:DIP-16_W7.62mm_Socket_LongPads"
+		(property "Footprint" "Package_DIP:DIP-16_W7.62mm_LongPads"
 			(at 92.456 64.77 0)
 			(effects
@@
 			)
 		)
-		(property "Footprint" "Package_DIP:DIP-16_W7.62mm_Socket_LongPads"
+		(property "Footprint" "Package_DIP:DIP-16_W7.62mm_LongPads"
 			(at 171.196 158.75 0)
 			(effects
@@
 			)
 		)
-		(property "Footprint" "Package_DIP:DIP-16_W7.62mm_Socket_LongPads"
+		(property "Footprint" "Package_DIP:DIP-16_W7.62mm_LongPads"
 			(at 171.196 140.97 0)
 			(effects
@@
 			)
 		)
-		(property "Footprint" "Package_DIP:DIP-16_W7.62mm_Socket_LongPads"
+		(property "Footprint" "Package_DIP:DIP-16_W7.62mm_LongPads"
 			(at 327.406 154.178 0)
 			(effects
