File: ram.kicad_sch (KiCad schematic)
At the start: 25 parts, among them U16 SIMM, U17 74LS08, U18 74LS74, U19 74F00, U32 74LS139, U34 74LS244, U35 74LS244

Commit message: - some IC are not socketed anymore to fit under shield
- updated logo
- silkscreen cleanup
- added pin1 indicator to solder jumpers
Parts:
- U17, U18, U19: footprint Package_DIP:DIP-14_W7.62mm_Socket_LongPads -> Package_DIP:DIP-14_W7.62mm_LongPads
- U32: footprint Package_DIP:DIP-16_W7.62mm_Socket_LongPads -> Package_DIP:DIP-16_W7.62mm_LongPads
- U34, U35: footprint Package_DIP:DIP-20_W7.62mm_Socket_LongPads -> Package_DIP:DIP-20_W7.62mm_LongPads
Changed lines of the file:
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@@
 			)
 		)
-		(property "Footprint" "Package_DIP:DIP-16_W7.62mm_Socket_LongPads"
+		(property "Footprint" "Package_DIP:DIP-16_W7.62mm_LongPads"
 			(at 139.7 193.04 0)
 			(effects
@@
 			)
 		)
-		(property "Footprint" "Package_DIP:DIP-16_W7.62mm_Socket_LongPads"
+		(property "Footprint" "Package_DIP:DIP-16_W7.62mm_LongPads"
 			(at 139.7 215.9 0)
 			(effects
@@
 			)
 		)
-		(property "Footprint" "Package_DIP:DIP-20_W7.62mm_Socket_LongPads"
+		(property "Footprint" "Package_DIP:DIP-20_W7.62mm_LongPads"
 			(at 78.74 93.98 0)
 			(effects
@@
 			)
 		)
-		(property "Footprint" "Package_DIP:DIP-14_W7.62mm_Socket_LongPads"
+		(property "Footprint" "Package_DIP:DIP-14_W7.62mm_LongPads"
 			(at 281.94 134.62 0)
 			(effects
@@
 			)
 		)
-		(property "Footprint" "Package_DIP:DIP-14_W7.62mm_Socket_LongPads"
+		(property "Footprint" "Package_DIP:DIP-14_W7.62mm_LongPads"
 			(at 281.94 149.86 0)
 			(effects
@@
 			)
 		)
-		(property "Footprint" "Package_DIP:DIP-14_W7.62mm_Socket_LongPads"
+		(property "Footprint" "Package_DIP:DIP-14_W7.62mm_LongPads"
 			(at 302.26 170.18 0)
 			(effects
@@
 			)
 		)
-		(property "Footprint" "Package_DIP:DIP-20_W7.62mm_Socket_LongPads"
+		(property "Footprint" "Package_DIP:DIP-20_W7.62mm_LongPads"
 			(at 78.74 53.34 0)
 			(effects
@@
 			)
 		)
-		(property "Footprint" "Package_DIP:DIP-14_W7.62mm_Socket_LongPads"
+		(property "Footprint" "Package_DIP:DIP-14_W7.62mm_LongPads"
 			(at 327.66 167.64 0)
 			(effects
@@
 			)
 		)
-		(property "Footprint" "Package_DIP:DIP-14_W7.62mm_Socket_LongPads"
+		(property "Footprint" "Package_DIP:DIP-14_W7.62mm_LongPads"
 			(at 39.37 109.22 0)
 			(effects
@@
 			)
 		)
-		(property "Footprint" "Package_DIP:DIP-14_W7.62mm_Socket_LongPads"
+		(property "Footprint" "Package_DIP:DIP-14_W7.62mm_LongPads"
 			(at 83.82 195.58 0)
 			(effects
@@
 			)
 		)
-		(property "Footprint" "Package_DIP:DIP-14_W7.62mm_Socket_LongPads"
+		(property "Footprint" "Package_DIP:DIP-14_W7.62mm_LongPads"
 			(at 293.37 226.06 0)
 			(effects
@@
 			)
 		)
-		(property "Footprint" "Package_DIP:DIP-14_W7.62mm_Socket_LongPads"
+		(property "Footprint" "Package_DIP:DIP-14_W7.62mm_LongPads"
 			(at 60.96 193.04 0)
 			(effects
@@
 			)
 		)
-		(property "Footprint" "Package_DIP:DIP-14_W7.62mm_Socket_LongPads"
+		(property "Footprint" "Package_DIP:DIP-14_W7.62mm_LongPads"
 			(at 327.66 137.16 0)
 			(effects
@@
 			)
 		)
-		(property "Footprint" "Package_DIP:DIP-14_W7.62mm_Socket_LongPads"
+		(property "Footprint" "Package_DIP:DIP-14_W7.62mm_LongPads"
 			(at 327.66 226.06 0)
 			(effects
@@
 			)
 		)
-		(property "Footprint" "Package_DIP:DIP-14_W7.62mm_Socket_LongPads"
+		(property "Footprint" "Package_DIP:DIP-14_W7.62mm_LongPads"
 			(at 361.95 226.06 0)
 			(effects
@@
 			)
 		)
-		(property "Footprint" "Package_DIP:DIP-14_W7.62mm_Socket_LongPads"
+		(property "Footprint" "Package_DIP:DIP-14_W7.62mm_LongPads"
 			(at 302.26 154.94 0)
 			(effects
@@
 			)
 		)
-		(property "Footprint" "Package_DIP:DIP-14_W7.62mm_Socket_LongPads"
+		(property "Footprint" "Package_DIP:DIP-14_W7.62mm_LongPads"
 			(at 214.63 80.01 0)
 			(effects

Commit message: Started cleaning up BOM
Other:
- company: SukkoPera -> Mathesar
Changed lines of the file:
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@@
 		(date "2026-04-09")
 		(rev "3")
-		(company "SukkoPera")
+		(company "Mathesar")
 		(comment 1 "OH NO! MATHESAR ADDED EVEN MORE STUFF TO REMEMBER")
 		(comment 2 "MEMORY AND...WELL, I USED TO REMEMBER")

Commit message: Working on BOM
Parts:
- C16, C17, C21: MFG Part Num C412C334M5U5TA -> C410C103K1R5TA; Mouser (none) -> 80-C410C103K1R
- C18, C19, C20: MFG Part Num C412C334M5U5TA -> C440C334K5R5TA7200; Mouser (none) -> 80-C440C334K5R-TR

Commit message: more work on BOM done
Parts:
- R201, R204, R205: MFG Name (none) -> YAGEO; MFG Part Num (none) -> MFR-25FBF52-4K7; Mouser (none) -> 603-MFR-25FBF52-4K7
- R206, R207, R208, R209, R210: MFG Name (none) -> YAGEO; MFG Part Num (none) -> MFR-25FBF52-68R; Mouser (none) -> 603-MFR-25FBF52-68R
Changed lines of the file:
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@@
 			)
 		)
-		(property "Mouser" ""
+		(property "Mouser" "603-MFR-25FBF52-4K7 "
+			(at 209.55 48.26 90)
+			(effects
+				(font
+					(size 1.27 1.27)
+				)
+				(hide yes)
+			)
+		)
+		(property "MFG Name" "YAGEO"
+			(at 209.55 48.26 90)
+			(effects
+				(font
+					(size 1.27 1.27)
+				)
+				(hide yes)
+			)
+		)
+		(property "MFG Part Num" "MFR-25FBF52-4K7 "
 			(at 209.55 48.26 90)
 			(effects
@@
 			)
 		)
-		(property "Mouser" ""
+		(property "Mouser" "603-MFR-25FBF52-68R "
+			(at 341.63 167.64 90)
+			(effects
+				(font
+					(size 1.27 1.27)
+				)
+				(hide yes)
+			)
+		)
+		(property "MFG Name" "YAGEO"
+			(at 341.63 167.64 90)
+			(effects
+				(font
+					(size 1.27 1.27)
+				)
+				(hide yes)
+			)
+		)
+		(property "MFG Part Num" "MFR-25FBF52-68R "
 			(at 341.63 167.64 90)
 			(effects
@@
 			)
 		)
-		(property "Mouser" ""
+		(property "Mouser" "603-MFR-25FBF52-4K7 "
+			(at 250.19 83.82 90)
+			(effects
+				(font
+					(size 1.27 1.27)
+				)
+				(hide yes)
+			)
+		)
+		(property "MFG Name" "YAGEO"
+			(at 250.19 83.82 90)
+			(effects
+				(font
+					(size 1.27 1.27)
+				)
+				(hide yes)
+			)
+		)
+		(property "MFG Part Num" "MFR-25FBF52-4K7 "
 			(at 250.19 83.82 90)
 			(effects
@@
 			)
 		)
-		(property "Mouser" ""
+		(property "Mouser" "603-MFR-25FBF52-68R "
+			(at 168.91 220.98 90)
+			(effects
+				(font
+					(size 1.27 1.27)
+				)
+				(hide yes)
+			)
+		)
+		(property "MFG Name" "YAGEO"
+			(at 168.91 220.98 90)
+			(effects
+				(font
+					(size 1.27 1.27)
+				)
+				(hide yes)
+			)
+		)
+		(property "MFG Part Num" "MFR-25FBF52-68R "
 			(at 168.91 220.98 90)
 			(effects
@@
 			)
 		)
-		(property "Mouser" ""
+		(property "Mouser" "603-MFR-25FBF52-68R "
+			(at 168.91 175.26 90)
+			(effects
+				(font
+					(size 1.27 1.27)
+				)
+				(hide yes)
+			)
+		)
+		(property "MFG Name" "YAGEO"
+			(at 168.91 175.26 90)
+			(effects
+				(font
+					(size 1.27 1.27)
+				)
+				(hide yes)
+			)
+		)
+		(property "MFG Part Num" "MFR-25FBF52-68R "
 			(at 168.91 175.26 90)
 			(effects
@@
 			)
 		)
-		(property "Mouser" ""
+		(property "Mouser" "603-MFR-25FBF52-4K7 "
+			(at 209.55 53.34 90)
+			(effects
+				(font
+					(size 1.27 1.27)
+				)
+				(hide yes)
+			)
+		)
+		(property "MFG Name" "YAGEO"
+			(at 209.55 53.34 90)
+			(effects
+				(font
+					(size 1.27 1.27)
+				)
+				(hide yes)
+			)
+		)
+		(property "MFG Part Num" "MFR-25FBF52-4K7 "
 			(at 209.55 53.34 90)
 			(effects
@@
 			)
 		)
-		(property "Mouser" ""
+		(property "Mouser" "603-MFR-25FBF52-68R "
+			(at 168.91 198.12 90)
+			(effects
+				(font
+					(size 1.27 1.27)
+				)
+				(hide yes)
+			)
+		)
+		(property "MFG Name" "YAGEO"
+			(at 168.91 198.12 90)
+			(effects
+				(font
+					(size 1.27 1.27)
+				)
+				(hide yes)
+			)
+		)
+		(property "MFG Part Num" "MFR-25FBF52-68R "
 			(at 168.91 198.12 90)
 			(effects
@@
 			)
 		)
-		(property "Mouser" ""
+		(property "Mouser" "603-MFR-25FBF52-68R "
+			(at 341.63 137.16 90)
+			(effects
+				(font
+					(size 1.27 1.27)
+				)
+				(hide yes)
+			)
+		)
+		(property "MFG Name" "YAGEO"
+			(at 341.63 137.16 90)
+			(effects
+				(font
+					(size 1.27 1.27)
+				)
+				(hide yes)
+			)
+		)
+		(property "MFG Part Num" "MFR-25FBF52-68R "
 			(at 341.63 137.16 90)
 			(effects

Commit message: More BOM work
I am marking optional components as DNP to get some overview
Parts:
- U16: MFG Name (none) -> TE CONNECTIVITY; MFG Part Num (none) -> 5822134-3; Mouser (none) -> 571-5822134-3
Changed lines of the file:
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@@
 			)
 		)
-		(property "Mouser" ""
+		(property "Mouser" "571-5822134-3 "
+			(at 247.65 226.06 0)
+			(effects
+				(font
+					(size 1.27 1.27)
+				)
+				(hide yes)
+			)
+		)
+		(property "MFG Name" "TE CONNECTIVITY"
+			(at 247.65 226.06 0)
+			(effects
+				(font
+					(size 1.27 1.27)
+				)
+				(hide yes)
+			)
+		)
+		(property "MFG Part Num" "5822134-3"
 			(at 247.65 226.06 0)
 			(effects
@@
 			)
 		)
-		(property "Mouser" ""
+		(property "Mouser" "571-5822134-3 "
 			(at 294.64 73.66 0)
 			(effects
+				(font
+					(size 1.27 1.27)
+				)
+				(hide yes)
+			)
+		)
+		(property "MFG Name" "TE CONNECTIVITY"
+			(at 294.64 73.66 0)
+			(effects
+				(font
+					(size 1.27 1.27)
+				)
+				(hide yes)
+			)
+		)
+		(property "MFG Part Num" "5822134-3"
+			(at 294.64 73.66 0)
+			(effects

Commit message: BOM updates
Parts:
- RP201, RP202, RP203: MFG Name (none) -> BOURNS; MFG Part Num (none) -> 4610X-102-680LF; Mouser (none) -> 652-4610X-2LF-68
- U17: MFG Name (none) -> TI; MFG Part Num (none) -> SN74LS08N; Mouser (none) -> 595-SN74LS08N
- U18: MFG Name (none) -> TI; MFG Part Num (none) -> SN74LS74AN; Mouser (none) -> 595-SN74LS74AN
- U19: MFG Name (none) -> TI; MFG Part Num (none) -> SN74F00N; Mouser (none) -> 595-SN74F00N
- U32: MFG Part Num SN74LS139AN -> SN74LS139AN; Mouser (none) -> 595-SN74LS139AN
- U34: MFG Name (none) -> TI; MFG Part Num (none) -> SN74LS244N; Mouser (none) -> 595-SN74LS244N
- U35: MFG Part Num SN74LS244N -> SN74LS244N; Mouser (none) -> 595-SN74LS244N
