File: ram.kicad_sch (KiCad schematic)
At the start: 25 parts, among them U16 SIMM, U17 74LS08, U18 74LS74, U19 74F00, U32 74LS139, U34 74LS244, U35 74LS244

Commit message: even  more BOM work
Parts:
- U17: value 74LS08 -> 74F08; MFG Part Num SN74LS08N -> SN74F08N; Mouser 595-SN74LS08N -> 595-SN74F08N
- U18: value 74LS74 -> 74F74; MFG Part Num SN74LS74AN -> SN74F74N; Mouser 595-SN74LS74AN -> 595-SN74F74N
- U32: value 74LS139 -> 74F139; MFG Part Num SN74LS139AN -> CD74ACT139E; Mouser 595-SN74LS139AN -> 595-CD74ACT139E
- U34, U35: value 74LS244 -> 74F244; MFG Part Num SN74LS244N -> (none); Mouser 595-SN74LS244N -> (none)
Changed lines of the file:
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@@
 			)
 		)
-		(property "Value" "74LS139"
+		(property "Value" "74F139"
 			(at 139.7 186.0296 0)
 			(effects
@@
 			)
 		)
-		(property "MFG Part Num" "SN74LS139AN "
+		(property "MFG Part Num" "CD74ACT139E "
 			(at 139.7 193.04 0)
 			(effects
@@
 			)
 		)
-		(property "Mouser" "595-SN74LS139AN "
+		(property "Mouser" "595-CD74ACT139E "
 			(at 139.7 193.04 0)
 			(effects
@@
 			)
 		)
-		(property "Value" "74LS139"
+		(property "Value" "74F139"
 			(at 139.7 208.8896 0)
 			(effects
@@
 			)
 		)
-		(property "MFG Part Num" "SN74LS139AN "
+		(property "MFG Part Num" "CD74ACT139E "
 			(at 139.7 215.9 0)
 			(effects
@@
 			)
 		)
-		(property "Mouser" "595-SN74LS139AN "
+		(property "Mouser" "595-CD74ACT139E "
 			(at 139.7 215.9 0)
 			(effects
@@
 			)
 		)
-		(property "Value" "74LS244"
+		(property "Value" "74F244"
 			(at 78.74 77.47 0)
 			(effects
@@
 			)
 		)
-		(property "MFG Part Num" "SN74LS244N "
+		(property "MFG Part Num" ""
 			(at 78.74 93.98 0)
 			(effects
@@
 			)
 		)
-		(property "Mouser" "595-SN74LS244N "
+		(property "Mouser" ""
 			(at 78.74 93.98 0)
 			(effects
@@
 			)
 		)
-		(property "Value" "74LS08"
+		(property "Value" "74F08"
 			(at 281.9317 143.51 0)
 			(effects
@@
 			)
 		)
-		(property "Mouser" "595-SN74LS08N "
+		(property "Mouser" "595-SN74F08N "
 			(at 281.94 149.86 0)
 			(effects
@@
 			)
 		)
-		(property "MFG Part Num" "SN74LS08N "
+		(property "MFG Part Num" "SN74F08N "
 			(at 281.94 149.86 0)
 			(effects
@@
 			)
 		)
-		(property "Value" "74LS08"
+		(property "Value" "74F08"
 			(at 302.2517 163.83 0)
 			(effects
@@
 			)
 		)
-		(property "Mouser" "595-SN74LS08N "
+		(property "Mouser" "595-SN74F08N "
 			(at 302.26 170.18 0)
 			(effects
@@
 			)
 		)
-		(property "MFG Part Num" "SN74LS08N "
+		(property "MFG Part Num" "SN74F08N "
 			(at 302.26 170.18 0)
 			(effects
@@
 			)
 		)
-		(property "Value" "74LS244"
+		(property "Value" "74F244"
 			(at 78.74 36.83 0)
 			(effects
@@
 			)
 		)
-		(property "Mouser" "595-SN74LS244N "
+		(property "Mouser" ""
 			(at 78.74 53.34 0)
 			(effects
@@
 			)
 		)
-		(property "MFG Part Num" "SN74LS244N "
+		(property "MFG Part Num" ""
 			(at 78.74 53.34 0)
 			(effects
@@
 			)
 		)
-		(property "Value" "74LS08"
+		(property "Value" "74F08"
 			(at 39.37 117.475 0)
 			(effects
@@
 			)
 		)
-		(property "Mouser" "595-SN74LS08N "
+		(property "Mouser" "595-SN74F08N "
 			(at 39.37 109.22 0)
 			(effects
@@
 			)
 		)
-		(property "MFG Part Num" "SN74LS08N "
+		(property "MFG Part Num" "SN74F08N "
 			(at 39.37 109.22 0)
 			(effects
@@
 			)
 		)
-		(property "Value" "74LS74"
+		(property "Value" "74F74"
 			(at 85.9633 187.96 0)
 			(effects
@@
 			)
 		)
-		(property "Mouser" "595-SN74LS74AN "
+		(property "Mouser" "595-SN74F74N "
 			(at 83.82 195.58 0)
 			(effects
@@
 			)
 		)
-		(property "MFG Part Num" "SN74LS74AN "
+		(property "MFG Part Num" "SN74F74N "
 			(at 83.82 195.58 0)
 			(effects
@@
 			)
 		)
-		(property "Value" "74LS74"
+		(property "Value" "74F74"
 			(at 299.72 227.3299 0)
 			(effects
@@
 			)
 		)
-		(property "Mouser" "595-SN74LS74AN "
+		(property "Mouser" "595-SN74F74N "
 			(at 293.37 226.06 0)
 			(effects
@@
 			)
 		)
-		(property "MFG Part Num" "SN74LS74AN "
+		(property "MFG Part Num" "SN74F74N "
 			(at 293.37 226.06 0)
 			(effects
@@
 			)
 		)
-		(property "Value" "74LS08"
+		(property "Value" "74F08"
 			(at 60.9517 186.69 0)
 			(effects
@@
 			)
 		)
-		(property "Mouser" "595-SN74LS08N "
+		(property "Mouser" "595-SN74F08N "
 			(at 60.96 193.04 0)
 			(effects
@@
 			)
 		)
-		(property "MFG Part Num" "SN74LS08N "
+		(property "MFG Part Num" "SN74F08N "
 			(at 60.96 193.04 0)
 			(effects
@@
 			)
 		)
-		(property "Value" "74LS08"
+		(property "Value" "74F08"
 			(at 334.01 227.3299 0)
 			(effects
@@
 			)
 		)
-		(property "Mouser" "595-SN74LS08N "
+		(property "Mouser" "595-SN74F08N "
 			(at 327.66 226.06 0)
 			(effects
@@
 			)
 		)
-		(property "MFG Part Num" "SN74LS08N "
+		(property "MFG Part Num" "SN74F08N "
 			(at 327.66 226.06 0)
 			(effects
@@
 			)
 		)
-		(property "Value" "74LS74"
+		(property "Value" "74F74"
 			(at 216.7733 72.39 0)
 			(effects
@@
 			)
 		)
-		(property "Mouser" "595-SN74LS74AN "
+		(property "Mouser" "595-SN74F74N "
 			(at 214.63 80.01 0)
 			(effects
@@
 			)
 		)
-		(property "MFG Part Num" "SN74LS74AN "
+		(property "MFG Part Num" "SN74F74N "
 			(at 214.63 80.01 0)
 			(effects

Commit message: added mouser part numbers
Parts:
- U34, U35: MFG Part Num (none) -> SN74F244N; Mouser (none) -> 595-SN74F244N
Changed lines of the file:
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@@
 			)
 		)
-		(property "MFG Part Num" ""
+		(property "MFG Part Num" "SN74F244N "
 			(at 78.74 93.98 0)
 			(effects
@@
 			)
 		)
-		(property "Mouser" ""
+		(property "Mouser" "595-SN74F244N "
 			(at 78.74 93.98 0)
 			(effects
@@
 			)
 		)
-		(property "Mouser" ""
+		(property "Mouser" "595-SN74F244N "
 			(at 78.74 53.34 0)
 			(effects
@@
 			)
 		)
-		(property "MFG Part Num" ""
+		(property "MFG Part Num" "SN74F244N "
 			(at 78.74 53.34 0)
 			(effects
