File: floppy.kicad_sch (KiCad schematic)
At the start: 25 parts, among them CN11 INTERNAL_FLOPPY, CN12 FLOPPY_POWER, CN14 IDE_POWER, CN15 IDE_I/F, CN5 EXTFLOPPY_DB23F, U36 74LS05, U5 GARY_5719

Commit message: DRAM chips replaced with SIMM module
Added logic to decode 2MB chip + 1.5MB slow
Rewired trapdoor slot
Other:
- title: Rämixx500 -> Rämixx500_max
Changed lines of the file:
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@@
 	(paper "A4")
 	(title_block
-		(title "Rämixx500")
-		(date "2019-06-23")
-		(rev "1")
+		(title "Rämixx500_max")
+		(date "2026-03-13")
+		(rev "2")
 		(company "SukkoPera")
 		(comment 1 "FLOPPY STUFF")

Commit message: Working on BOM
Parts:
- CN14, CN15: now not fitted
- CN5: MFG Name (none) -> COMMODORE; MFG Part Num (none) -> 390241-03

Commit message: More BOM work
I am marking optional components as DNP to get some overview
Parts:
- E601, E602: Mouser (none) -> 81-DSS1NB32A103Q91A
- E611, E612, E613, E614, E615, E616, E617, E618, E619, E620, E621, E622, E623, E624, E625, E626: MFG Name (none) -> MURATA; MFG Part Num DSS1NB32A101Q91A (has ferrite) -> DSS1NB32A101Q91A; Mouser (none) -> 81-DSS1NB32A101Q91A
- U5: MFG Name (none) -> COMMODORE
Changed lines of the file:
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@@
 			)
 		)
-		(property "MFG Part Num" "DSS1NB32A101Q91A (has ferrite)"
+		(property "MFG Part Num" "DSS1NB32A101Q91A "
 			(at 74.549 141.224 0)
 			(effects
@@
 			)
 		)
-		(property "Mouser" ""
+		(property "Mouser" "81-DSS1NB32A101Q91A "
+			(at 74.549 141.224 0)
+			(effects
+				(font
+					(size 1.27 1.27)
+				)
+				(hide yes)
+			)
+		)
+		(property "MFG Name" "MURATA"
 			(at 74.549 141.224 0)
 			(effects
@@
 			)
 		)
-		(property "MFG Part Num" "DSS1NB32A101Q91A (has ferrite)"
+		(property "MFG Part Num" "DSS1NB32A101Q91A "
 			(at 84.328 146.304 0)
 			(effects
@@
 			)
 		)
-		(property "Mouser" ""
+		(property "Mouser" "81-DSS1NB32A101Q91A "
+			(at 84.328 146.304 0)
+			(effects
+				(font
+					(size 1.27 1.27)
+				)
+				(hide yes)
+			)
+		)
+		(property "MFG Name" "MURATA"
 			(at 84.328 146.304 0)
 			(effects
@@
 			)
 		)
-		(property "MFG Part Num" "DSS1NB32A101Q91A (has ferrite)"
+		(property "MFG Part Num" "DSS1NB32A101Q91A "
 			(at 74.549 151.384 0)
 			(effects
@@
 			)
 		)
-		(property "Mouser" ""
+		(property "Mouser" "81-DSS1NB32A101Q91A "
+			(at 74.549 151.384 0)
+			(effects
+				(font
+					(size 1.27 1.27)
+				)
+				(hide yes)
+			)
+		)
+		(property "MFG Name" "MURATA"
 			(at 74.549 151.384 0)
 			(effects
@@
 			)
 		)
-		(property "MFG Part Num" "DSS1NB32A101Q91A (has ferrite)"
+		(property "MFG Part Num" "DSS1NB32A101Q91A "
 			(at 84.328 156.464 0)
 			(effects
@@
 			)
 		)
-		(property "Mouser" ""
+		(property "Mouser" "81-DSS1NB32A101Q91A "
+			(at 84.328 156.464 0)
+			(effects
+				(font
+					(size 1.27 1.27)
+				)
+				(hide yes)
+			)
+		)
+		(property "MFG Name" "MURATA"
 			(at 84.328 156.464 0)
 			(effects
@@
 			)
 		)
-		(property "Mouser" ""
+		(property "Mouser" "81-DSS1NB32A103Q91A "
 			(at 74.549 161.544 0)
 			(effects
@@
 			)
 		)
-		(property "MFG Part Num" "DSS1NB32A101Q91A (has ferrite)"
+		(property "MFG Part Num" "DSS1NB32A101Q91A "
 			(at 74.549 105.664 0)
 			(effects
@@
 			)
 		)
-		(property "Mouser" ""
+		(property "Mouser" "81-DSS1NB32A101Q91A "
+			(at 74.549 105.664 0)
+			(effects
+				(font
+					(size 1.27 1.27)
+				)
+				(hide yes)
+			)
+		)
+		(property "MFG Name" "MURATA"
 			(at 74.549 105.664 0)
 			(effects
@@
 			)
 		)
-		(property "MFG Part Num" "DSS1NB32A101Q91A (has ferrite)"
+		(property "MFG Part Num" "DSS1NB32A101Q91A "
 			(at 84.328 110.744 0)
 			(effects
@@
 			)
 		)
-		(property "Mouser" ""
+		(property "Mouser" "81-DSS1NB32A101Q91A "
+			(at 84.328 110.744 0)
+			(effects
+				(font
+					(size 1.27 1.27)
+				)
+				(hide yes)
+			)
+		)
+		(property "MFG Name" "MURATA"
 			(at 84.328 110.744 0)
 			(effects
@@
 			)
 		)
-		(property "MFG Part Num" "DSS1NB32A101Q91A (has ferrite)"
+		(property "MFG Part Num" "DSS1NB32A101Q91A "
 			(at 136.017 108.204 0)
 			(effects
@@
 			)
 		)
-		(property "Mouser" ""
+		(property "Mouser" "81-DSS1NB32A101Q91A "
+			(at 136.017 108.204 0)
+			(effects
+				(font
+					(size 1.27 1.27)
+				)
+				(hide yes)
+			)
+		)
+		(property "MFG Name" "MURATA"
 			(at 136.017 108.204 0)
 			(effects
@@
 			)
 		)
-		(property "MFG Part Num" "DSS1NB32A101Q91A (has ferrite)"
+		(property "MFG Part Num" "DSS1NB32A101Q91A "
 			(at 126.238 113.284 0)
 			(effects
@@
 			)
 		)
-		(property "Mouser" ""
+		(property "Mouser" "81-DSS1NB32A101Q91A "
+			(at 126.238 113.284 0)
+			(effects
+				(font
+					(size 1.27 1.27)
+				)
+				(hide yes)
+			)
+		)
+		(property "MFG Name" "MURATA"
 			(at 126.238 113.284 0)
 			(effects
@@
 			)
 		)
-		(property "MFG Part Num" "DSS1NB32A101Q91A (has ferrite)"
+		(property "MFG Part Num" "DSS1NB32A101Q91A "
 			(at 136.017 118.364 0)
 			(effects
@@
 			)
 		)
-		(property "Mouser" ""
+		(property "Mouser" "81-DSS1NB32A101Q91A "
+			(at 136.017 118.364 0)
+			(effects
+				(font
+					(size 1.27 1.27)
+				)
+				(hide yes)
+			)
+		)
+		(property "MFG Name" "MURATA"
 			(at 136.017 118.364 0)
 			(effects
@@
 			)
 		)
-		(property "MFG Part Num" "DSS1NB32A101Q91A (has ferrite)"
+		(property "MFG Part Num" "DSS1NB32A101Q91A "
 			(at 126.238 123.444 0)
 			(effects
@@
 			)
 		)
-		(property "Mouser" ""
+		(property "Mouser" "81-DSS1NB32A101Q91A "
+			(at 126.238 123.444 0)
+			(effects
+				(font
+					(size 1.27 1.27)
+				)
+				(hide yes)
+			)
+		)
+		(property "MFG Name" "MURATA"
 			(at 126.238 123.444 0)
 			(effects
@@
 			)
 		)
-		(property "MFG Part Num" "DSS1NB32A101Q91A (has ferrite)"
+		(property "MFG Part Num" "DSS1NB32A101Q91A "
 			(at 136.017 128.524 0)
 			(effects
@@
 			)
 		)
-		(property "Mouser" ""
+		(property "Mouser" "81-DSS1NB32A101Q91A "
+			(at 136.017 128.524 0)
+			(effects
+				(font
+					(size 1.27 1.27)
+				)
+				(hide yes)
+			)
+		)
+		(property "MFG Name" "MURATA"
 			(at 136.017 128.524 0)
 			(effects
@@
 			)
 		)
-		(property "MFG Part Num" "DSS1NB32A101Q91A (has ferrite)"
+		(property "MFG Part Num" "DSS1NB32A101Q91A "
 			(at 126.238 133.604 0)
 			(effects
@@
 			)
 		)
-		(property "Mouser" ""
+		(property "Mouser" "81-DSS1NB32A101Q91A "
+			(at 126.238 133.604 0)
+			(effects
+				(font
+					(size 1.27 1.27)
+				)
+				(hide yes)
+			)
+		)
+		(property "MFG Name" "MURATA"
 			(at 126.238 133.604 0)
 			(effects
@@
 			)
 		)
-		(property "MFG Part Num" "DSS1NB32A101Q91A (has ferrite)"
+		(property "MFG Part Num" "DSS1NB32A101Q91A "
 			(at 136.017 138.684 0)
 			(effects
@@
 			)
 		)
-		(property "Mouser" ""
+		(property "Mouser" "81-DSS1NB32A101Q91A "
+			(at 136.017 138.684 0)
+			(effects
+				(font
+					(size 1.27 1.27)
+				)
+				(hide yes)
+			)
+		)
+		(property "MFG Name" "MURATA"
 			(at 136.017 138.684 0)
 			(effects
@@
 			)
 		)
-		(property "MFG Part Num" "DSS1NB32A101Q91A (has ferrite)"
+		(property "MFG Part Num" "DSS1NB32A101Q91A "
 			(at 126.238 143.764 0)
 			(effects
@@
 			)
 		)
-		(property "Mouser" ""
+		(property "Mouser" "81-DSS1NB32A101Q91A "
+			(at 126.238 143.764 0)
+			(effects
+				(font
+					(size 1.27 1.27)
+				)
+				(hide yes)
+			)
+		)
+		(property "MFG Name" "MURATA"
 			(at 126.238 143.764 0)
 			(effects
@@
 			)
 		)
-		(property "MFG Part Num" "DSS1NB32A101Q91A (has ferrite)"
+		(property "MFG Part Num" "DSS1NB32A101Q91A "
 			(at 136.017 148.844 0)
 			(effects
@@
 			)
 		)
-		(property "Mouser" ""
+		(property "Mouser" "81-DSS1NB32A101Q91A "
+			(at 136.017 148.844 0)
+			(effects
+				(font
+					(size 1.27 1.27)
+				)
+				(hide yes)
+			)
+		)
+		(property "MFG Name" "MURATA"
 			(at 136.017 148.844 0)
 			(effects
@@
 			)
 		)
-		(property "MFG Part Num" "DSS1NB32A101Q91A (has ferrite)"
+		(property "MFG Part Num" "DSS1NB32A101Q91A "
 			(at 126.238 153.924 0)
 			(effects
@@
 			)
 		)
-		(property "Mouser" ""
+		(property "Mouser" "81-DSS1NB32A101Q91A "
+			(at 126.238 153.924 0)
+			(effects
+				(font
+					(size 1.27 1.27)
+				)
+				(hide yes)
+			)
+		)
+		(property "MFG Name" "MURATA"
 			(at 126.238 153.924 0)
 			(effects
@@
 			)
 		)
-		(property "Mouser" ""
+		(property "Mouser" "81-DSS1NB32A103Q91A "
 			(at 136.017 159.004 0)
 			(effects
@@
 			(at 68.199 47.244 0)
 			(effects
+				(font
+					(size 1.27 1.27)
+				)
+				(hide yes)
+			)
+		)
+		(property "MFG Name" "COMMODORE"
+			(at 68.199 47.244 0)
+			(effects

Commit message: BOM updates
Parts:
- CN11: MFG Name (none) -> AMPHENOL; MFG Part Num (none) -> 77313-101-34LF; Mouser (none) -> 649-77313-101-34LF
- CN12: MFG Name (none) -> TE CONNECTIVITY; MFG Part Num (none) -> 171825-4; Mouser (none) -> 571-1718254
- U36: MFG Part Num SN74LS05N -> SN74LS05N; Mouser (none) -> 595-SN74LS05N
- U5: MFG Name COMMODORE -> 3M; MFG Part Num (none) -> 4848-6000-CP; Mouser (none) -> 517-4848-6000-CP
Changed lines of the file:
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@@
 			)
 		)
-		(property "Mouser" ""
+		(property "Mouser" "649-77313-101-34LF "
+			(at 175.641 57.15 0)
+			(effects
+				(font
+					(size 1.27 1.27)
+				)
+				(hide yes)
+			)
+		)
+		(property "MFG Name" "AMPHENOL"
+			(at 175.641 57.15 0)
+			(effects
+				(font
+					(size 1.27 1.27)
+				)
+				(hide yes)
+			)
+		)
+		(property "MFG Part Num" "77313-101-34LF "
 			(at 175.641 57.15 0)
 			(effects
@@
 			)
 		)
-		(property "Mouser" ""
+		(property "Mouser" "517-4848-6000-CP "
 			(at 68.199 47.244 0)
 			(effects
@@
 			)
 		)
-		(property "MFG Name" "COMMODORE"
+		(property "MFG Name" "3M"
+			(at 68.199 47.244 0)
+			(effects
+				(font
+					(size 1.27 1.27)
+				)
+				(hide yes)
+			)
+		)
+		(property "MFG Part Num" "4848-6000-CP "
 			(at 68.199 47.244 0)
 			(effects
@@
 			)
 		)
-		(property "MFG Part Num" "SN74LS05N"
+		(property "MFG Part Num" "SN74LS05N "
 			(at 100.076 39.624 0)
 			(effects
@@
 			)
 		)
-		(property "Mouser" ""
+		(property "Mouser" "595-SN74LS05N "
 			(at 100.076 39.624 0)
 			(effects
@@
 			)
 		)
-		(property "MFG Part Num" "SN74LS05N"
+		(property "MFG Part Num" "SN74LS05N "
 			(at 100.076 49.784 0)
 			(effects
@@
 			)
 		)
-		(property "Mouser" ""
+		(property "Mouser" "595-SN74LS05N "
 			(at 100.076 49.784 0)
 			(effects
@@
 			)
 		)
-		(property "MFG Part Num" "SN74LS05N"
+		(property "MFG Part Num" "SN74LS05N "
 			(at 100.076 59.944 0)
 			(effects
@@
 			)
 		)
-		(property "Mouser" ""
+		(property "Mouser" "595-SN74LS05N "
 			(at 100.076 59.944 0)
 			(effects
@@
 			)
 		)
-		(property "MFG Part Num" "SN74LS05N"
+		(property "MFG Part Num" "SN74LS05N "
 			(at 100.076 70.104 0)
 			(effects
@@
 			)
 		)
-		(property "Mouser" ""
+		(property "Mouser" "595-SN74LS05N "
 			(at 100.076 70.104 0)
 			(effects
@@
 			)
 		)
-		(property "Mouser" ""
+		(property "Mouser" "571-1718254 "
+			(at 241.3 62.865 0)
+			(effects
+				(font
+					(size 1.27 1.27)
+				)
+				(hide yes)
+			)
+		)
+		(property "MFG Name" "TE CONNECTIVITY"
+			(at 241.3 62.865 0)
+			(effects
+				(font
+					(size 1.27 1.27)
+				)
+				(hide yes)
+			)
+		)
+		(property "MFG Part Num" "171825-4 "
 			(at 241.3 62.865 0)
 			(effects

Commit message: replaced commodore hybrid with OpenAmigaVideoHybrid
decided to place address pullups for better EPROM capability
Parts:
- CN11: MFG Name AMPHENOL -> ADAM TECH; MFG Part Num 77313-101-34LF -> BHR-34-VUA; Mouser 649-77313-101-34LF -> 737-BHR-34-VUA
Changed lines of the file:
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@@
 			)
 		)
-		(property "Mouser" "649-77313-101-34LF "
+		(property "Mouser" "737-BHR-34-VUA "
 			(at 175.641 57.15 0)
 			(effects
@@
 			)
 		)
-		(property "MFG Name" "AMPHENOL"
+		(property "MFG Name" "ADAM TECH"
 			(at 175.641 57.15 0)
 			(effects
@@
 			)
 		)
-		(property "MFG Part Num" "77313-101-34LF "
+		(property "MFG Part Num" "BHR-34-VUA"
 			(at 175.641 57.15 0)
 			(effects
