File: floppy.kicad_sch (KiCad schematic)
At the start: 25 parts, among them CN11 INTERNAL_FLOPPY, CN12 FLOPPY_POWER, CN14 IDE_POWER, CN15 IDE_I/F, CN5 EXTFLOPPY_DB23F, U36 74LS05, U5 GARY_5719

Commit message: added pin 1 indications like on originnal board
changed floppy connector to non-shrouded version
Parts:
- CN11: MFG Name ADAM TECH -> AMPHENOL; MFG Part Num BHR-34-VUA -> 77313-101-34LF; Mouser 737-BHR-34-VUA -> 649-77313-101-34LF
Changed lines of the file:
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@@
 			)
 		)
-		(property "Mouser" "737-BHR-34-VUA "
+		(property "Mouser" "649-77313-101-34LF"
 			(at 175.641 57.15 0)
 			(effects
@@
 			)
 		)
-		(property "MFG Name" "ADAM TECH"
+		(property "MFG Name" "AMPHENOL"
 			(at 175.641 57.15 0)
 			(effects
@@
 			)
 		)
-		(property "MFG Part Num" "BHR-34-VUA"
+		(property "MFG Part Num" "77313-101-34LF"
 			(at 175.641 57.15 0)
 			(effects

Commit message: more silkscreen work
removed sockets for standard IC's
Parts:
- CN11: footprint Connector_IDC:IDC-Header_2x17_P2.54mm_Vertical -> Connector_PinHeader_2.54mm:PinHeader_2x17_P2.54mm_Vertical
- U36: footprint Package_DIP:DIP-14_W7.62mm_Socket_LongPads -> Package_DIP:DIP-14_W7.62mm_LongPads
Changed lines of the file:
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@@
 	(title_block
 		(title "Rämixx500_max")
-		(date "2026-04-09")
+		(date "2026-04-26")
 		(rev "3")
 		(company "SukkoPera")
@@
 			)
 		)
-		(property "Footprint" "Connector_IDC:IDC-Header_2x17_P2.54mm_Vertical"
+		(property "Footprint" "Connector_PinHeader_2.54mm:PinHeader_2x17_P2.54mm_Vertical"
 			(at 175.641 57.15 0)
 			(effects
@@
 			)
 		)
-		(property "Footprint" "Package_DIP:DIP-14_W7.62mm_Socket_LongPads"
+		(property "Footprint" "Package_DIP:DIP-14_W7.62mm_LongPads"
 			(at 100.076 39.624 0)
 			(effects
@@
 			)
 		)
-		(property "Footprint" "Package_DIP:DIP-14_W7.62mm_Socket_LongPads"
+		(property "Footprint" "Package_DIP:DIP-14_W7.62mm_LongPads"
 			(at 100.076 49.784 0)
 			(effects
@@
 			)
 		)
-		(property "Footprint" "Package_DIP:DIP-14_W7.62mm_Socket_LongPads"
+		(property "Footprint" "Package_DIP:DIP-14_W7.62mm_LongPads"
 			(at 100.076 59.944 0)
 			(effects
@@
 			)
 		)
-		(property "Footprint" "Package_DIP:DIP-14_W7.62mm_Socket_LongPads"
+		(property "Footprint" "Package_DIP:DIP-14_W7.62mm_LongPads"
 			(at 100.076 70.104 0)
 			(effects
