File: Raemixx500.kicad_pcb (KiCad board)
At the start: 2 copper layers, 365.8 x 254 mm, 372 parts, among them CN1 LEFT_JOY, CN10 COMPOSITE, CN11 INTERNAL_FLOPPY, CN12 FLOPPY_POWER, CN13 KEYBOARD, CN14 IDE_POWER, CN15 IDE_I/F, CN2 RIGHT_JOY, CN3 RIGHT, CN4 LEFT, CN5 EXTFLOPPY_DB23F, CN6 SERIAL_DB25M, CN7 PARALLEL_DB25F, CN8 POWER, CN9 VIDEO_DB23M, J90 DRIVE_SWITCHER, J91 Dispatcher_3to1, J92 Dispatcher_3to1, J93 Dispatcher_3to1, J99 HD_ACT, P1 EXPANSION BUS, P9 TRAPDOOR, Q301 2N3906, Q321 MPF102 / J113, Q331 MPF102 / J113, Q501 2N3904, Q502 2N3906, Q503 2N3906, Q504 2N3904, Q711 2N3904, Q921 MMBFJ113, Q931 MMBFJ113, U1 68000D, U10 74LS244, U11 74LS373, U12 74LS244, U13 74LS373, U14 LF347, U15 74LS157, U16 SIMM, U17 74F08, U18 74F74, U19 74F00, U2 FAT_AGNUS_8375, U3 PAULA, U32 74F139, U33 74F258, U34 74F244, U35 74F244, U36 74LS05, U37 74LS32, U38 MC1488, U39 MC1489, U4 DENISE, U40 74HCT245, U41 74HCT245, U42 NE555, U5 GARY_5719, U6 ROM, U7 VIA_8520, U8 VIA_8520, U9 MSM6242B, U94 74HCT14, X1 XTAL, Y9 32.768kHz

Commit message: more silkscreen work
removed sockets for standard IC's
Parts:
- CN11: footprint Connector_IDC:IDC-Header_2x17_P2.54mm_Vertical -> Connector_PinHeader_2.54mm:PinHeader_2x17_P2.54mm_Vertical
- U10, U11, U12, U13, U40, U41: footprint Package_DIP:DIP-20_W7.62mm_Socket_LongPads -> Package_DIP:DIP-20_W7.62mm_LongPads
- U14, U36, U37, U38, U39: footprint Package_DIP:DIP-14_W7.62mm_Socket_LongPads -> Package_DIP:DIP-14_W7.62mm_LongPads
- U15, U33: footprint Package_DIP:DIP-16_W7.62mm_Socket_LongPads -> Package_DIP:DIP-16_W7.62mm_LongPads
- U42: footprint Package_DIP:DIP-8_W7.62mm_Socket_LongPads -> Package_DIP:DIP-8_W7.62mm_LongPads
