File: Raemixx500.kicad_sch (KiCad schematic)
At the start: 3 parts

Commit message: DRAM chips replaced with SIMM module
Added logic to decode 2MB chip + 1.5MB slow
Rewired trapdoor slot
Other:
- title: Rämixx500 -> Rämixx500_max
Changed lines of the file:
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@@
 	(paper "A4")
 	(title_block
-		(title "Rämixx500")
-		(date "2021-05-26")
-		(rev "1")
+		(title "Rämixx500_max")
+		(date "2026-03-13")
+		(rev "2")
 		(company "SukkoPera")
 		(comment 4 "Licensed under CC BY-NC-SA 4.0")

Commit message: - some IC are not socketed anymore to fit under shield
- updated logo
- silkscreen cleanup
- added pin1 indicator to solder jumpers
Parts:
- V2: footprint Raemixx500:Logo -> Raemixx500:logo_max
Changed lines of the file:
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@@
 			)
 		)
-		(property "Footprint" "Raemixx500:Logo"
+		(property "Footprint" "Raemixx500:logo_max"
 			(at 162.052 182.88 0)
 			(effects

Commit message: Started cleaning up BOM
Parts:
- V0, V1, V2: now left out of the parts list
Changed lines of the file:
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@@
 		(unit 1)
 		(exclude_from_sim no)
-		(in_bom yes)
+		(in_bom no)
 		(on_board yes)
 		(dnp no)
@@
 		(unit 1)
 		(exclude_from_sim no)
-		(in_bom yes)
+		(in_bom no)
 		(on_board yes)
 		(dnp no)
@@
 		(unit 1)
 		(exclude_from_sim no)
-		(in_bom yes)
+		(in_bom no)
 		(on_board yes)
 		(dnp no)
