File: rom.kicad_sch (KiCad schematic)
At the start: 5 parts, among them J91 Dispatcher_3to1, J92 Dispatcher_3to1, J93 Dispatcher_3to1, U6 ROM

Commit message: DRAM chips replaced with SIMM module
Added logic to decode 2MB chip + 1.5MB slow
Rewired trapdoor slot
Other:
- title: Rämixx500 -> Rämixx500_max
Changed lines of the file:
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@@
 	(paper "A4")
 	(title_block
-		(title "Rämixx500")
-		(date "2019-04-20")
-		(rev "1")
+		(title "Rämixx500_max")
+		(date "2026-03-13")
+		(rev "2")
 		(company "SukkoPera")
 		(comment 4 "Licensed under CC BY-NC-SA 4.0")

Commit message: Working on BOM
Parts:
- C6: MFG Part Num C412C334M5U5TA -> C440C334K5R5TA7200; Mouser (none) -> 80-C440C334K5R-TR
- J91, J92, J93: now not fitted
Changed lines of the file:
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@@
+			)
+		)
+		(property "Mouser" ""
+			(at 168.656 91.313 0)
+			(effects
+				(font
+					(size 1.27 1.27)
+				)
+				(hide yes)
 			)
 		)
@@
 			)
 		)
+		(property "Mouser" ""
+			(at 244.348 91.313 0)
+			(effects
+				(font
+					(size 1.27 1.27)
+				)
+				(hide yes)
+			)
+		)
 		(pin "41"
 		)
@@
 			)
 		)
-		(property "MFG Part Num" "C412C334M5U5TA"
+		(property "MFG Part Num" "C440C334K5R5TA7200"
 			(at 264.795 90.297 0)
 			(effects
@@
 		)
 		(property "Required" "R"
+			(at 264.795 90.297 0)
+			(effects
+				(font
+					(size 1.27 1.27)
+				)
+				(hide yes)
+			)
+		)
+		(property "Mouser" "80-C440C334K5R-TR "
 			(at 264.795 90.297 0)
 			(effects
@@
 		(in_bom yes)
 		(on_board yes)
-		(dnp no)
+		(dnp yes)
 		(property "Reference" "J91"
 			(at 71.12 60.9092 0)
@@
 					(size 1.27 1.27)
 				)
+			)
+		)
+		(property "Mouser" ""
+			(at 69.85 68.961 0)
+			(effects
+				(font
+					(size 1.27 1.27)
+				)
+				(hide yes)
 			)
 		)
@@
 		(in_bom yes)
 		(on_board yes)
-		(dnp no)
+		(dnp yes)
 		(property "Reference" "J92"
 			(at 71.12 83.2612 0)
@@
 					(size 1.27 1.27)
 				)
+			)
+		)
+		(property "Mouser" ""
+			(at 69.85 91.313 0)
+			(effects
+				(font
+					(size 1.27 1.27)
+				)
+				(hide yes)
 			)
 		)
@@
 		(in_bom yes)
 		(on_board yes)
-		(dnp no)
+		(dnp yes)
 		(property "Reference" "J93"
 			(at 71.12 105.3592 0)
@@
 			)
 		)
+		(property "Mouser" ""
+			(at 69.85 113.411 0)
+			(effects
+				(font
+					(size 1.27 1.27)
+				)
+				(hide yes)
+			)
+		)

Commit message: BOM updates
Parts:
- U6: MFG Name (none) -> AMIGA/HYPERION
Changed lines of the file:
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@@
+			)
+		)
+		(property "MFG Name" "AMIGA/HYPERION"
+			(at 168.656 91.313 0)
+			(effects
+				(font
+					(size 1.27 1.27)
+				)
+				(hide yes)
 			)
 		)
@@
 			(at 244.348 91.313 0)
 			(effects
+				(font
+					(size 1.27 1.27)
+				)
+				(hide yes)
+			)
+		)
+		(property "MFG Name" "AMIGA/HYPERION"
+			(at 244.348 91.313 0)
+			(effects

Commit message: BOM work done
Parts:
- U6: MFG Name AMIGA/HYPERION -> 3M; MFG Part Num (none) -> 4842-6000-CP; Mouser (none) -> 517-4842-6000-CP
Changed lines of the file:
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@@
 			)
 		)
-		(property "Mouser" ""
+		(property "Mouser" "517-4842-6000-CP "
 			(at 168.656 91.313 0)
 			(effects
@@
 			)
 		)
-		(property "MFG Name" "AMIGA/HYPERION"
+		(property "MFG Name" "3M"
+			(at 168.656 91.313 0)
+			(effects
+				(font
+					(size 1.27 1.27)
+				)
+				(hide yes)
+			)
+		)
+		(property "MFG Part Num" "4842-6000-CP "
 			(at 168.656 91.313 0)
 			(effects
@@
 			)
 		)
-		(property "Mouser" ""
-			(at 244.348 91.313 0)
-			(effects
-				(font
-					(size 1.27 1.27)
-				)
-				(hide yes)
-			)
-		)
-		(property "MFG Name" "AMIGA/HYPERION"
-			(at 244.348 91.313 0)
-			(effects
+		(property "Mouser" "517-4842-6000-CP "
+			(at 244.348 91.313 0)
+			(effects
+				(font
+					(size 1.27 1.27)
+				)
+				(hide yes)
+			)
+		)
+		(property "MFG Name" "3M"
+			(at 244.348 91.313 0)
+			(effects
+				(font
+					(size 1.27 1.27)
+				)
+				(hide yes)
+			)
+		)
+		(property "MFG Part Num" "4842-6000-CP "
+			(at 244.348 91.313 0)
+			(effects
