File: cias.kicad_sch (KiCad schematic)
At the start: 69 parts, among them CN13 KEYBOARD, CN6 SERIAL_DB25M, CN7 PARALLEL_DB25F, J90 DRIVE_SWITCHER, J99 HD_ACT, Q501 2N3904, Q502 2N3906, Q503 2N3906, Q504 2N3904, Q711 2N3904, U38 MC1488, U39 MC1489, U42 NE555, U7 VIA_8520, U8 VIA_8520

Commit message: more work on BOM done
Parts:
- D501: MFG Name (none) -> ONSEMI; MFG Part Num (none) -> 1N4148TR; Mouser (none) -> 512-1N4148TR
- R109: MFG Name (none) -> YAGEO; MFG Part Num (none) -> MFR-25FBF52-68R; Mouser (none) -> 603-MFR-25FBF52-68R
- R501, R504, R505, R506, R509, R510: MFG Name (none) -> YAGEO; MFG Part Num (none) -> MFR-25FBF52-10K; Mouser (none) -> 603-MFR-25FBF52-10K
- R502: MFG Name (none) -> YAGEO; MFG Part Num (none) -> MFR-25FBF52-2K7; Mouser (none) -> 603-MFR-25FBF52-2K7
- R503, R508: MFG Name (none) -> YAGEO; MFG Part Num (none) -> MFR-25FBF52-4K7; Mouser (none) -> 603-MFR-25FBF52-4K7
- R507: MFG Name (none) -> YAGEO; MFG Part Num (none) -> MFR-25FBF52-100R; Mouser (none) -> 603-MFR-25FBF52-100R
- R711: MFG Name (none) -> YAGEO; MFG Part Num (none) -> MFR-25FBF52-1M; Mouser (none) -> 603-MFR-25FBF52-1M
- R712: MFG Name (none) -> YAGEO; MFG Part Num (none) -> MFR-25FBF52-47K; Mouser (none) -> 603-MFR-25FBF52-47K
- R713: MFG Name (none) -> YAGEO; MFG Part Num (none) -> MFR-25FBF52-1K; Mouser (none) -> 603-MFR-25FBF52-1K

Commit message: More BOM work
I am marking optional components as DNP to get some overview
Parts:
- E501, E502, E503: MFG Name (none) -> VISHAY; MFG Part Num (none) -> PR01000104709JA500; Mouser (none) -> 594-PR01000104709JA5
- E511, E512, E513, E514, E515, E516, E517, E518, E519, E521, E522, E523, E524, E631, E632: MFG Name (none) -> MURATA; MFG Part Num DSS1NB32A101Q91A (has ferrite) -> DSS1NB32A101Q91A; Mouser (none) -> 81-DSS1NB32A101Q91A
- E520, E531, E533, E535, E536, E537, E538: Mouser (none) -> 81-DSS1NB32A471Q91A
- E532, E534: Mouser (none) -> 81-DSS1NB32A151Q91A
- Q501, Q504, Q711: MFG Name (none) -> ONSEMI; MFG Part Num (none) -> 2N3904BU; Mouser (none) -> 512-2N3904BU
- Q502, Q503: MFG Name (none) -> ONSEMI; MFG Part Num (none) -> 2N3906BU; Mouser (none) -> 512-2N3906BU
- U7, U8: MFG Name (none) -> COMMODORE

Commit message: BOM updates
Parts:
- CN13: MFG Name (none) -> AMPHENOL; MFG Part Num (none) -> 10129378-908003BLF; Mouser (none) -> 649-1012937890803BLF
- J99: MFG Name (none) -> AMPHENOL; MFG Part Num (none) -> 10129378-902003BLF; Mouser (none) -> 649-1012937890203BLF
- RP501: MFG Name (none) -> BOURNS; MFG Part Num (none) -> 4610X-101-103LF; Mouser (none) -> 652-4610X-1LF-10K
- U38: MFG Part Num MC1488N -> SN75C188N; Mouser (none) -> 595-SN75C188N
- U39: MFG Part Num MC1489N -> SN75C189N; Mouser (none) -> 595-SN75C189N
- U42: MFG Part Num NE555P -> SA555P; Mouser (none) -> 595-SA555P
Changed lines of the file:
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@@
 			)
 		)
-		(property "Mouser" ""
+		(property "Mouser" "652-4610X-1LF-10K "
+			(at 146.05 88.646 0)
+			(effects
+				(font
+					(size 1.27 1.27)
+				)
+				(hide yes)
+			)
+		)
+		(property "MFG Name" "BOURNS"
+			(at 146.05 88.646 0)
+			(effects
+				(font
+					(size 1.27 1.27)
+				)
+				(hide yes)
+			)
+		)
+		(property "MFG Part Num" "4610X-101-103LF"
 			(at 146.05 88.646 0)
 			(effects
@@
 			)
 		)
-		(property "MFG Part Num" "MC1488N"
+		(property "MFG Part Num" "SN75C188N "
 			(at 184.15 167.894 0)
 			(effects
@@
 			)
 		)
-		(property "Mouser" ""
+		(property "Mouser" "595-SN75C188N "
 			(at 184.15 167.894 0)
 			(effects
@@
 			)
 		)
-		(property "MFG Part Num" "MC1488N"
+		(property "MFG Part Num" "SN75C188N "
 			(at 184.15 157.353 0)
 			(effects
@@
 			)
 		)
-		(property "Mouser" ""
+		(property "Mouser" "595-SN75C188N "
 			(at 184.15 157.353 0)
 			(effects
@@
 			)
 		)
-		(property "MFG Part Num" "MC1488N"
+		(property "MFG Part Num" "SN75C188N "
 			(at 184.15 178.054 0)
 			(effects
@@
 			)
 		)
-		(property "Mouser" ""
+		(property "Mouser" "595-SN75C188N "
 			(at 184.15 178.054 0)
 			(effects
@@
 			)
 		)
-		(property "MFG Part Num" "MC1489N"
+		(property "MFG Part Num" "SN75C189N "
 			(at 163.703 172.974 0)
 			(effects
@@
 			)
 		)
-		(property "Mouser" ""
+		(property "Mouser" "595-SN75C189N "
 			(at 163.703 172.974 0)
 			(effects
@@
 			)
 		)
-		(property "MFG Part Num" "MC1489N"
+		(property "MFG Part Num" "SN75C189N "
 			(at 154.686 188.214 0)
 			(effects
@@
 			)
 		)
-		(property "Mouser" ""
+		(property "Mouser" "595-SN75C189N "
 			(at 154.686 188.214 0)
 			(effects
@@
 			)
 		)
-		(property "MFG Part Num" "MC1489N"
+		(property "MFG Part Num" "SN75C189N "
 			(at 141.859 198.374 0)
 			(effects
@@
 			)
 		)
-		(property "Mouser" ""
+		(property "Mouser" "595-SN75C189N "
 			(at 141.859 198.374 0)
 			(effects
@@
 			)
 		)
-		(property "MFG Part Num" "MC1489N"
+		(property "MFG Part Num" "SN75C189N "
 			(at 141.859 183.134 0)
 			(effects
@@
 			)
 		)
-		(property "Mouser" ""
+		(property "Mouser" "595-SN75C189N "
 			(at 141.859 183.134 0)
 			(effects
@@
 			)
 		)
-		(property "MFG Part Num" "MC1489N"
+		(property "MFG Part Num" "SN75C189N "
 			(at 38.735 263.144 0)
 			(effects
@@
 			)
 		)
-		(property "Mouser" ""
+		(property "Mouser" "595-SN75C189N "
 			(at 38.735 263.144 0)
 			(effects
@@
 			)
 		)
-		(property "MFG Part Num" "MC1488N"
+		(property "MFG Part Num" "SN75C188N "
 			(at 54.991 263.144 0)
 			(effects
@@
 			)
 		)
-		(property "Mouser" ""
+		(property "Mouser" "595-SN75C188N "
 			(at 54.991 263.144 0)
 			(effects
@@
 			)
 		)
-		(property "Mouser" ""
+		(property "Mouser" "649-1012937890803BLF "
+			(at 382.27 80.01 0)
+			(effects
+				(font
+					(size 1.27 1.27)
+				)
+				(hide yes)
+			)
+		)
+		(property "MFG Name" "AMPHENOL"
+			(at 382.27 80.01 0)
+			(effects
+				(font
+					(size 1.27 1.27)
+				)
+				(hide yes)
+			)
+		)
+		(property "MFG Part Num" "10129378-908003BLF "
 			(at 382.27 80.01 0)
 			(effects
@@
 			)
 		)
-		(property "MFG Part Num" "NE555P"
+		(property "MFG Part Num" "SA555P "
 			(at 322.961 195.453 0)
 			(effects
@@
 			)
 		)
-		(property "Mouser" ""
+		(property "Mouser" "595-SA555P "
 			(at 322.961 195.453 0)
 			(effects
@@
 			)
 		)
-		(property "MFG Part Num" "NE555P"
+		(property "MFG Part Num" "SA555P "
 			(at 397.002 196.088 0)
 			(effects
@@
 			)
 		)
-		(property "Mouser" ""
+		(property "Mouser" "595-SA555P "
 			(at 397.002 196.088 0)
 			(effects
@@
 			)
 		)
-		(property "Mouser" ""
+		(property "Mouser" "649-1012937890203BLF "
+			(at 307.34 121.92 0)
+			(effects
+				(font
+					(size 1.27 1.27)
+				)
+				(hide yes)
+			)
+		)
+		(property "MFG Name" "AMPHENOL"
+			(at 307.34 121.92 0)
+			(effects
+				(font
+					(size 1.27 1.27)
+				)
+				(hide yes)
+			)
+		)
+		(property "MFG Part Num" "10129378-902003BLF "
 			(at 307.34 121.92 0)
 			(effects

Commit message: BOM work done
Parts:
- U7, U8: MFG Name COMMODORE -> 3M; MFG Part Num (none) -> 4840-6000-CP; Mouser (none) -> 517-4840-6000-CP
Changed lines of the file:
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@@
 			)
 		)
-		(property "Mouser" ""
+		(property "Mouser" "517-4840-6000-CP "
 			(at 84.201 87.884 0)
 			(effects
@@
 			)
 		)
-		(property "MFG Name" "COMMODORE"
+		(property "MFG Name" "3M"
+			(at 84.201 87.884 0)
+			(effects
+				(font
+					(size 1.27 1.27)
+				)
+				(hide yes)
+			)
+		)
+		(property "MFG Part Num" "4840-6000-CP "
 			(at 84.201 87.884 0)
 			(effects
@@
 			)
 		)
-		(property "Mouser" ""
+		(property "Mouser" "517-4840-6000-CP "
 			(at 84.201 160.655 0)
 			(effects
@@
 			)
 		)
-		(property "MFG Name" "COMMODORE"
+		(property "MFG Name" "3M"
+			(at 84.201 160.655 0)
+			(effects
+				(font
+					(size 1.27 1.27)
+				)
+				(hide yes)
+			)
+		)
+		(property "MFG Part Num" "4840-6000-CP "
 			(at 84.201 160.655 0)
 			(effects
@@
 			)
 		)
-		(property "Mouser" ""
+		(property "Mouser" "517-4840-6000-CP "
 			(at 159.004 260.604 0)
 			(effects
@@
 			)
 		)
-		(property "MFG Name" "COMMODORE"
+		(property "MFG Name" "3M"
+			(at 159.004 260.604 0)
+			(effects
+				(font
+					(size 1.27 1.27)
+				)
+				(hide yes)
+			)
+		)
+		(property "MFG Part Num" "4840-6000-CP "
 			(at 159.004 260.604 0)
 			(effects
@@
 			)
 		)
-		(property "Mouser" ""
+		(property "Mouser" "517-4840-6000-CP "
 			(at 194.945 260.604 0)
 			(effects
@@
 			)
 		)
-		(property "MFG Name" "COMMODORE"
+		(property "MFG Name" "3M"
 			(at 194.945 260.604 0)
 			(effects
+				(font
+					(size 1.27 1.27)
+				)
+				(hide yes)
+			)
+		)
+		(property "MFG Part Num" "4840-6000-CP "
+			(at 194.945 260.604 0)
+			(effects

Commit message: more silkscreen work
removed sockets for standard IC's
Parts:
- U38, U39: footprint Package_DIP:DIP-14_W7.62mm_Socket_LongPads -> Package_DIP:DIP-14_W7.62mm_LongPads
- U42: footprint Package_DIP:DIP-8_W7.62mm_Socket_LongPads -> Package_DIP:DIP-8_W7.62mm_LongPads
Changed lines of the file:
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@@
 	(title_block
 		(title "Rämixx500_max")
-		(date "2026-04-09")
+		(date "2026-04-26")
 		(rev "3")
 		(company "SukkoPera")
@@
 			)
 		)
-		(property "Footprint" "Package_DIP:DIP-14_W7.62mm_Socket_LongPads"
+		(property "Footprint" "Package_DIP:DIP-14_W7.62mm_LongPads"
 			(at 184.15 174.244 0)
 			(effects
@@
 			)
 		)
-		(property "Footprint" "Package_DIP:DIP-14_W7.62mm_Socket_LongPads"
+		(property "Footprint" "Package_DIP:DIP-14_W7.62mm_LongPads"
 			(at 184.15 163.703 0)
 			(effects
@@
 			)
 		)
-		(property "Footprint" "Package_DIP:DIP-14_W7.62mm_Socket_LongPads"
+		(property "Footprint" "Package_DIP:DIP-14_W7.62mm_LongPads"
 			(at 184.15 184.404 0)
 			(effects
@@
 			)
 		)
-		(property "Footprint" "Package_DIP:DIP-14_W7.62mm_Socket_LongPads"
+		(property "Footprint" "Package_DIP:DIP-14_W7.62mm_LongPads"
 			(at 163.703 179.324 0)
 			(effects
@@
 			)
 		)
-		(property "Footprint" "Package_DIP:DIP-14_W7.62mm_Socket_LongPads"
+		(property "Footprint" "Package_DIP:DIP-14_W7.62mm_LongPads"
 			(at 154.686 194.564 0)
 			(effects
@@
 			)
 		)
-		(property "Footprint" "Package_DIP:DIP-14_W7.62mm_Socket_LongPads"
+		(property "Footprint" "Package_DIP:DIP-14_W7.62mm_LongPads"
 			(at 141.859 204.724 0)
 			(effects
@@
 			)
 		)
-		(property "Footprint" "Package_DIP:DIP-14_W7.62mm_Socket_LongPads"
+		(property "Footprint" "Package_DIP:DIP-14_W7.62mm_LongPads"
 			(at 141.859 189.484 0)
 			(effects
@@
 			)
 		)
-		(property "Footprint" "Package_DIP:DIP-14_W7.62mm_Socket_LongPads"
+		(property "Footprint" "Package_DIP:DIP-14_W7.62mm_LongPads"
 			(at 38.735 269.494 0)
 			(effects
@@
 			)
 		)
-		(property "Footprint" "Package_DIP:DIP-14_W7.62mm_Socket_LongPads"
+		(property "Footprint" "Package_DIP:DIP-14_W7.62mm_LongPads"
 			(at 54.991 269.494 0)
 			(effects
@@
 			)
 		)
-		(property "Footprint" "Package_DIP:DIP-8_W7.62mm_Socket_LongPads"
+		(property "Footprint" "Package_DIP:DIP-8_W7.62mm_LongPads"
 			(at 322.961 195.453 0)
 			(effects
@@
 			)
 		)
-		(property "Footprint" "Package_DIP:DIP-8_W7.62mm_Socket_LongPads"
+		(property "Footprint" "Package_DIP:DIP-8_W7.62mm_LongPads"
 			(at 397.002 196.088 0)
 			(effects
