File: cpu.kicad_sch (KiCad schematic)
At the start: 25 parts, among them U1 68000D, U10 74LS244, U11 74LS373, U12 74LS244, U13 74LS373, U2 FAT_AGNUS_8375, U33 74LS258, U37 74LS32, U5 GARY_5719, X1 XTAL

Commit message: BOM updates
Parts:
- U1: MFG Name MOTOROLA -> MILL-MAX; MFG Part Num (none) -> 110-93-964-41-001000; Mouser (none) -> 575-193964
- U10, U12: MFG Part Num SN74LS244N -> SN74LS244N; Mouser (none) -> 595-SN74LS244N
- U11, U13: Mouser (none) -> 595-SN74LS373N
- U2: MFG Name COMMODORE -> MILL-MAX; MFG Part Num (none) -> 940-44-084-24-000000; Mouser (none) -> 575-948424
- U33: MFG Name N/A -> TI; MFG Part Num (none) -> SN74LS258BN; Mouser (none) -> 595-SN74LS258BN
- U37: MFG Part Num SN74LS32N -> SN74LS32N; Mouser (none) -> 595-SN74LS32N
- U5: MFG Name COMMODORE -> 3M; MFG Part Num (none) -> 4848-6000-CP; Mouser (none) -> 517-4848-6000-CP
Changed lines of the file:
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@@
 			)
 		)
-		(property "Mouser" ""
+		(property "Mouser" "575-948424 "
 			(at 291.592 190.119 0)
 			(effects
@@
 			)
 		)
-		(property "MFG Name" "COMMODORE"
+		(property "MFG Name" "MILL-MAX"
+			(at 291.592 190.119 0)
+			(effects
+				(font
+					(size 1.27 1.27)
+				)
+				(hide yes)
+			)
+		)
+		(property "MFG Part Num" "940-44-084-24-000000 "
 			(at 291.592 190.119 0)
 			(effects
@@
 			)
 		)
-		(property "MFG Part Num" "SN74LS32N"
+		(property "MFG Part Num" "SN74LS32N "
 			(at 335.28 104.648 0)
 			(effects
@@
 			)
 		)
-		(property "Mouser" ""
+		(property "Mouser" "595-SN74LS32N "
 			(at 335.28 104.648 0)
 			(effects
@@
 			)
 		)
-		(property "MFG Part Num" "SN74LS32N"
+		(property "MFG Part Num" "SN74LS32N "
 			(at 335.28 113.157 0)
 			(effects
@@
 			)
 		)
-		(property "Mouser" ""
+		(property "Mouser" "595-SN74LS32N "
 			(at 335.28 113.157 0)
 			(effects
@@
 			)
 		)
-		(property "MFG Name" "N/A"
+		(property "MFG Name" "TI"
 			(at 218.694 260.604 0)
 			(effects
@@
 			)
 		)
-		(property "Mouser" ""
+		(property "Mouser" "595-SN74LS258BN "
+			(at 218.694 260.604 0)
+			(effects
+				(font
+					(size 1.27 1.27)
+				)
+				(hide yes)
+			)
+		)
+		(property "MFG Part Num" "SN74LS258BN"
 			(at 218.694 260.604 0)
 			(effects
@@
 			)
 		)
-		(property "Mouser" ""
+		(property "Mouser" "575-193964 "
 			(at 92.329 117.729 0)
 			(effects
@@
 			)
 		)
-		(property "MFG Name" "MOTOROLA"
+		(property "MFG Name" "MILL-MAX"
+			(at 92.329 117.729 0)
+			(effects
+				(font
+					(size 1.27 1.27)
+				)
+				(hide yes)
+			)
+		)
+		(property "MFG Part Num" "110-93-964-41-001000"
 			(at 92.329 117.729 0)
 			(effects
@@
 			)
 		)
-		(property "Mouser" ""
+		(property "Mouser" "595-SN74LS373N "
 			(at 172.085 97.409 90)
 			(effects
@@
 			)
 		)
-		(property "Mouser" ""
+		(property "Mouser" "595-SN74LS373N "
 			(at 172.085 168.529 90)
 			(effects
@@
 			)
 		)
-		(property "MFG Part Num" "SN74LS244N"
+		(property "MFG Part Num" "SN74LS244N "
 			(at 172.085 132.842 0)
 			(effects
@@
 			)
 		)
-		(property "Mouser" ""
+		(property "Mouser" "595-SN74LS244N "
 			(at 172.085 132.842 90)
 			(effects
@@
 			)
 		)
-		(property "MFG Part Num" "SN74LS244N"
+		(property "MFG Part Num" "SN74LS244N "
 			(at 172.085 61.595 0)
 			(effects
@@
 			)
 		)
-		(property "Mouser" ""
+		(property "Mouser" "595-SN74LS244N "
 			(at 172.085 61.595 90)
 			(effects
@@
 			)
 		)
-		(property "Mouser" ""
+		(property "Mouser" "517-4848-6000-CP "
+			(at 291.592 62.23 0)
+			(effects
+				(font
+					(size 1.27 1.27)
+				)
+				(hide yes)
+			)
+		)
+		(property "MFG Name" "3M"
 			(at 291.592 62.23 0)
 			(effects
@@
 			)
 		)
-		(property "MFG Name" "COMMODORE"
+		(property "MFG Part Num" "4848-6000-CP "
 			(at 291.592 62.23 0)
 			(effects

Commit message: even  more BOM work
Parts:
- C99: now not fitted
- U33: value 74LS258 -> 74F258; MFG Part Num SN74LS258BN -> (none); Mouser 595-SN74LS258BN -> (none)
Changed lines of the file:
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@@
 			)
 		)
-		(property "Value" "74LS258"
+		(property "Value" "74F258"
 			(at 219.329 254.6604 0)
 			(effects
@@
 			)
 		)
-		(property "Mouser" "595-SN74LS258BN "
-			(at 218.694 260.604 0)
-			(effects
-				(font
-					(size 1.27 1.27)
-				)
-				(hide yes)
-			)
-		)
-		(property "MFG Part Num" "SN74LS258BN"
+		(property "Mouser" ""
+			(at 218.694 260.604 0)
+			(effects
+				(font
+					(size 1.27 1.27)
+				)
+				(hide yes)
+			)
+		)
+		(property "MFG Part Num" ""
 			(at 218.694 260.604 0)
 			(effects
@@
 		(in_bom yes)
 		(on_board yes)
-		(dnp no)
+		(dnp yes)
 		(property "Reference" "C99"
 			(at 370.586 217.6526 0)

Commit message: added mouser part numbers
Parts:
- U33: MFG Part Num (none) -> SN74F258N; Mouser (none) -> 595-SN74F258N
Changed lines of the file:
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@@
 			)
 		)
-		(property "Mouser" ""
+		(property "Mouser" "595-SN74F258N "
 			(at 218.694 260.604 0)
 			(effects
@@
 			)
 		)
-		(property "MFG Part Num" ""
+		(property "MFG Part Num" "SN74F258N "
 			(at 218.694 260.604 0)
 			(effects

Commit message: more silkscreen work
removed sockets for standard IC's
Parts:
- U10, U11, U12, U13: footprint Package_DIP:DIP-20_W7.62mm_Socket_LongPads -> Package_DIP:DIP-20_W7.62mm_LongPads
- U33: footprint Package_DIP:DIP-16_W7.62mm_Socket_LongPads -> Package_DIP:DIP-16_W7.62mm_LongPads
- U37: footprint Package_DIP:DIP-14_W7.62mm_Socket_LongPads -> Package_DIP:DIP-14_W7.62mm_LongPads
Changed lines of the file:
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@@
 	(title_block
 		(title "Rämixx500_max")
-		(date "2026-04-09")
+		(date "2026-04-26")
 		(rev "3")
 		(company "SukkoPera")
@@
 			)
 		)
-		(property "Footprint" "Package_DIP:DIP-14_W7.62mm_Socket_LongPads"
+		(property "Footprint" "Package_DIP:DIP-14_W7.62mm_LongPads"
 			(at 335.28 104.648 0)
 			(effects
@@
 			)
 		)
-		(property "Footprint" "Package_DIP:DIP-14_W7.62mm_Socket_LongPads"
+		(property "Footprint" "Package_DIP:DIP-14_W7.62mm_LongPads"
 			(at 335.28 113.157 0)
 			(effects
@@
 			)
 		)
-		(property "Footprint" "Package_DIP:DIP-16_W7.62mm_Socket_LongPads"
+		(property "Footprint" "Package_DIP:DIP-16_W7.62mm_LongPads"
 			(at 297.434 319.024 0)
 			(effects
@@
 			)
 		)
-		(property "Footprint" "Package_DIP:DIP-20_W7.62mm_Socket_LongPads"
+		(property "Footprint" "Package_DIP:DIP-20_W7.62mm_LongPads"
 			(at 172.085 97.409 0)
 			(effects
@@
 			)
 		)
-		(property "Footprint" "Package_DIP:DIP-20_W7.62mm_Socket_LongPads"
+		(property "Footprint" "Package_DIP:DIP-20_W7.62mm_LongPads"
 			(at 172.085 168.529 0)
 			(effects
@@
 			)
 		)
-		(property "Footprint" "Package_DIP:DIP-20_W7.62mm_Socket_LongPads"
+		(property "Footprint" "Package_DIP:DIP-20_W7.62mm_LongPads"
 			(at 172.085 132.842 0)
 			(effects
@@
 			)
 		)
-		(property "Footprint" "Package_DIP:DIP-20_W7.62mm_Socket_LongPads"
+		(property "Footprint" "Package_DIP:DIP-20_W7.62mm_LongPads"
 			(at 172.085 61.595 0)
 			(effects
