File: rtc.kicad_sch (KiCad schematic)
At the start: 16 parts, among them U36 74LS05, U9 MSM6242B, Y9 32.768kHz

Commit message: BOM work done
Parts:
- U9: MFG Name (none) -> 3M; MFG Part Num (none) -> 4818-3000-CP; Mouser (none) -> 517-4818-3000-CP
Changed lines of the file:
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@@
 			)
 		)
-		(property "Mouser" ""
+		(property "Mouser" "517-4818-3000-CP "
+			(at 203.073 53.975 0)
+			(effects
+				(font
+					(size 1.27 1.27)
+				)
+				(hide yes)
+			)
+		)
+		(property "MFG Name" "3M"
+			(at 203.073 53.975 0)
+			(effects
+				(font
+					(size 1.27 1.27)
+				)
+				(hide yes)
+			)
+		)
+		(property "MFG Part Num" "4818-3000-CP "
 			(at 203.073 53.975 0)
 			(effects
@@
 			)
 		)
-		(property "Mouser" ""
+		(property "Mouser" "517-4818-3000-CP "
 			(at 115.697 147.955 0)
 			(effects
+				(font
+					(size 1.27 1.27)
+				)
+				(hide yes)
+			)
+		)
+		(property "MFG Name" "3M"
+			(at 115.697 147.955 0)
+			(effects
+				(font
+					(size 1.27 1.27)
+				)
+				(hide yes)
+			)
+		)
+		(property "MFG Part Num" "4818-3000-CP "
+			(at 115.697 147.955 0)
+			(effects

Commit message: more silkscreen work
removed sockets for standard IC's
Parts:
- BT9: MFG Name Eagle Plastic Devices -> EAGLE PLASTIC DEVICES
- TC9: MFG Name JML06-1 -> (none)
- U36: footprint Package_DIP:DIP-14_W7.62mm_Socket_LongPads -> Package_DIP:DIP-14_W7.62mm_LongPads
Changed lines of the file:
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@@
 	(title_block
 		(title "Rämixx500_max")
-		(date "2026-04-09")
+		(date "2026-04-26")
 		(rev "3")
 		(company "SukkoPera")
@@
 			)
 		)
-		(property "Footprint" "Package_DIP:DIP-14_W7.62mm_Socket_LongPads"
+		(property "Footprint" "Package_DIP:DIP-14_W7.62mm_LongPads"
 			(at 118.872 64.135 0)
 			(effects
@@
 			)
 		)
-		(property "MFG Name" "JML06-1"
+		(property "MFG Name" ""
 			(at 244.856 59.055 90)
 			(effects
@@
 			)
 		)
-		(property "Footprint" "Package_DIP:DIP-14_W7.62mm_Socket_LongPads"
+		(property "Footprint" "Package_DIP:DIP-14_W7.62mm_LongPads"
 			(at 80.518 64.135 0)
 			(effects
@@
 			)
 		)
-		(property "MFG Name" "Eagle Plastic Devices"
+		(property "MFG Name" "EAGLE PLASTIC DEVICES"
 			(at 74.93 149.098 0)
 			(effects
