File: trapdoor.kicad_sch (KiCad schematic)
At the start: 2 parts, among them P9 TRAPDOOR

Commit message: BOM updates
Parts:
- P9: MFG Name (none) -> ADAM TECH; MFG Part Num (none) -> PH2RA-80-UA; Mouser (none) -> 737-PH2RA-80-UA
Changed lines of the file:
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@@
 			)
 		)
-		(property "Mouser" ""
+		(property "Mouser" "737-PH2RA-80-UA "
 			(at 156.21 95.25 0)
 			(effects
+				(font
+					(size 1.27 1.27)
+				)
+				(hide yes)
+			)
+		)
+		(property "MFG Name" "ADAM TECH"
+			(at 156.21 95.25 0)
+			(effects
+				(font
+					(size 1.27 1.27)
+				)
+				(hide yes)
+			)
+		)
+		(property "MFG Part Num" "PH2RA-80-UA "
+			(at 156.21 95.25 0)
+			(effects
